Commit message: (feat): add simulation with Ignition

File: gripper_pincette/description/ros2_control/gripper_pincette.ros2_control.xacro (robot description, xacro)
@@ -1,6 +1,6 @@
 <?xml version="1.0"?>
 <robot xmlns:xacro="http://www.ros.org/wiki/xacro">
-  <xacro:macro name="gripper_pincette_ros2_control" params="name use_gazebo_classic:=^|false">
-    <ros2_control name="${name}" type="system">
+  <xacro:macro name="gripper_pincette_ros2_control" params="name">
+  <ros2_control name="${name}" type="system">
     <hardware>
       <plugin>gazebo_ros2_control/GazeboSystem</plugin>

File: gripper_pincette/description/urdf/gripper_pincette_ign.urdf.xacro (robot description, xacro)
@@ -3,5 +3,5 @@
   <xacro:include filename="$(find gripper_pincette)/description/urdf/gripper_pincette_description.urdf.xacro" />
   <!-- Import gripper_pincette ros2_control description -->
-  <xacro:include filename="$(find gripper_pincette)/description/ros2_control/gripper_pincette.ros2_control.xacro" />
+  <xacro:include filename="$(find gripper_pincette)/description/ros2_control/gripper_pincette_ign.ros2_control.xacro" />
   <xacro:gripper_pincette/>
   <!-- create link fixed to the "world" -->
@@ -14,6 +14,6 @@
     <axis xyz="0 0 1"/>
   </joint>
-  <xacro:gripper_pincette_ros2_control name="gripper_pincette"/>
-  <xacro:include filename="$(find gripper_pincette)/description/gazebo/gripper_pincette.gazebo.xacro" />
-  <xacro:gripper_pincette_gazebo/>
+  <xacro:gripper_pincette_ros2_control_ign name="gripper_pincette"/>
+  <xacro:include filename="$(find gripper_pincette)/description/gazebo/gripper_pincette_ign.gazebo.xacro" />
+  <xacro:gripper_pincette_gazebo_ign/>
 </robot>
