Commit message: (fix): use ignition only

File: explorer/description/gazebo/explorer.gazebo.xacro (robot description, xacro)
@@ -1,15 +1,116 @@
 <?xml version="1.0"?>
-<!--
-Copied and modified from ROS1 example -
-https://github.com/ros-simulation/gazebo_ros_demos/blob/kinetic-devel/rrbot_description/urdf/rrbot.gazebo
--->
 <robot xmlns:xacro="http://ros.org/wiki/xacro">
   <xacro:macro name="explorer_gazebo" params="">
     <!-- ros_control plugin -->
     <gazebo>
-      <plugin filename="libgazebo_ros2_control.so" name="gazebo_ros2_control_explorer">
+      <plugin filename="libign_ros2_control-system.so" name="ign_ros2_control::IgnitionROS2ControlPlugin">
         <parameters>$(find ros2_control_explorer)/config/explorer_controller.yaml</parameters>
       </plugin>
     </gazebo>
+    <gazebo reference="base_link">
+      <visual>
+          <material>
+              <diffuse>1 1 1 1</diffuse>
+          </material>
+      </visual>
+    </gazebo>
+    <gazebo reference="link_1">
+      <visual>
+          <material>
+              <diffuse>1 1 1 1</diffuse>
+          </material>
+      </visual>
+    </gazebo>
+    <gazebo reference="link_2">
+      <visual>
+          <material>
+              <diffuse>1 1 1 1</diffuse>
+          </material>
+      </visual>
+    </gazebo>
+    <gazebo reference="link_3">
+      <visual>
+          <material>
+              <diffuse>1 1 1 1</diffuse>
+          </material>
+      </visual>
+    </gazebo>
+    <gazebo reference="link_4">
+      <visual>
+          <material>
+              <diffuse>1 1 1 1</diffuse>
+          </material>
+      </visual>
+    </gazebo>
+    <gazebo reference="link_5">
+      <visual>
+          <material>
+              <diffuse>1 1 1 1</diffuse>
+          </material>
+      </visual>
+    </gazebo>
+    <gazebo reference="structure">
+      <visual>
+          <material>
+              <diffuse>1 1 1 1</diffuse>
+          </material>
+      </visual>
+    </gazebo>
+    <gazebo reference="motor">
+      <visual>
+          <material>
+              <diffuse>1 1 1 1</diffuse>
+          </material>
+      </visual>
+    </gazebo>
+    <gazebo reference="palm_top_shell">
+      <visual>
+          <material>
+              <diffuse>1 1 1 1</diffuse>
+          </material>
+      </visual>
+    </gazebo>
+    <gazebo reference="right_finger_first_phalanx">
+      <visual>
+          <material>
+              <diffuse>1 1 1 1</diffuse>
+          </material>
+      </visual>
+    </gazebo>
+    <gazebo reference="right_external_rod">
+      <visual>
+          <material>
+              <diffuse>1 1 1 1</diffuse>
+          </material>
+      </visual>
+    </gazebo>
+    <gazebo reference="right_finger_last_phalanx">
+      <visual>
+          <material>
+              <diffuse>1 1 1 1</diffuse>
+          </material>
+      </visual>
+    </gazebo>
+    <gazebo reference="left_finger_first_phalanx">
+      <visual>
+          <material>
+              <diffuse>1 1 1 1</diffuse>
+          </material>
+      </visual>
+    </gazebo>
+    <gazebo reference="left_external_rod">
+      <visual>
+          <material>
+              <diffuse>1 1 1 1</diffuse>
+          </material>
+      </visual>
+    </gazebo>
+    <gazebo reference="left_finger_last_phalanx">
+      <visual>
+          <material>
+              <diffuse>1 1 1 1</diffuse>
+          </material>
+      </visual>
+    </gazebo>
   </xacro:macro>
 </robot>

File: explorer/description/ros2_control/explorer.ros2_control.xacro (robot description, xacro)
@@ -1,11 +1,11 @@
 <?xml version="1.0"?>
 <robot xmlns:xacro="http://www.ros.org/wiki/xacro">
-  <xacro:macro name="explorer_ros2_control" params="name use_gazebo_classic:=^|false">
+  <xacro:macro name="explorer_ros2_control" params="name use_ignition:=^|false">
     <ros2_control name="${name}" type="system">
       <hardware>
-        <xacro:if value="${use_gazebo_classic}">
-          <plugin>gazebo_ros2_control/GazeboSystem</plugin>
+        <xacro:if value="${use_ignition}">
+          <plugin>ign_ros2_control/IgnitionSystem</plugin>
         </xacro:if>
-        <xacro:unless value="${use_gazebo_classic}">
+        <xacro:unless value="${use_ignition}">
           <plugin>ros2_control_explorer/RobotSystem</plugin>
         </xacro:unless>
@@ -99,4 +99,5 @@
         <state_interface name="position"/>
         <state_interface name="velocity"/>
+        <state_interface name="effort"/>
       </joint>
       <joint name="right_external_rod_joint">
@@ -106,4 +107,5 @@
         <state_interface name="position"/>
         <state_interface name="velocity"/>
+        <state_interface name="effort"/>
       </joint>
       <joint name="right_fingertip_joint">
@@ -113,4 +115,5 @@
         <state_interface name="position"/>
         <state_interface name="velocity"/>
+        <state_interface name="effort"/>
       </joint>
       <joint name="left_finger_joint">
@@ -120,4 +123,5 @@
         <state_interface name="position"/>
         <state_interface name="velocity"/>
+        <state_interface name="effort"/>
       </joint>
       <joint name="left_external_rod_joint">
@@ -127,4 +131,5 @@
         <state_interface name="position"/>
         <state_interface name="velocity"/>
+        <state_interface name="effort"/>
       </joint>
       <joint name="left_fingertip_joint">
@@ -134,4 +139,5 @@
         <state_interface name="position"/>
         <state_interface name="velocity"/>
+        <state_interface name="effort"/>
       </joint>
     </ros2_control>

File: explorer/description/urdf/explorer.urdf.xacro (robot description, xacro)
@@ -1,5 +1,5 @@
 <?xml version="1.0"?>
 <robot xmlns:xacro="http://wiki.ros.org/xacro" name="explorer">
-  <xacro:arg name="use_gazebo_classic" default="false" />
+  <xacro:arg name="use_ignition" default="false" />
   <!-- Import explorer macro -->
   <xacro:include filename="$(find ros2_control_explorer)/description/urdf/explorer_old_description.urdf.xacro"/>
@@ -35,7 +35,7 @@
   <!-- Import explorer ros2_control description -->
   <xacro:include filename="$(find ros2_control_explorer)/description/ros2_control/explorer.ros2_control.xacro" />
-  <xacro:explorer_ros2_control name="explorer" use_gazebo_classic="$(arg use_gazebo_classic)"/>
-  <xacro:if value="$(arg use_gazebo_classic)">
-    <!-- Import Gazebo Classic definitions + plugin -->
+  <xacro:explorer_ros2_control name="explorer" use_ignition="$(arg use_ignition)"/>
+  <xacro:if value="$(arg use_ignition)">
+    <!-- Import Ignition definitions + plugin -->
     <xacro:include filename="$(find ros2_control_explorer)/description/gazebo/explorer.gazebo.xacro" />
     <xacro:explorer_gazebo/>

File: gripper_pincette/description/gazebo/gripper_pincette.gazebo.xacro (robot description, xacro)
@@ -8,8 +8,71 @@
     <!-- ros_control plugin -->
     <gazebo>
-      <plugin filename="libgazebo_ros2_control.so" name="gazebo_ros2_control_gripper_pincette">
+       <plugin filename="ign_ros2_control-system" name="ign_ros2_control::IgnitionROS2ControlPlugin">
         <parameters>$(find gripper_pincette)/config/gripper_controller.yaml</parameters>
       </plugin>
     </gazebo>
+    <gazebo reference="structure">
+      <visual>
+          <material>
+              <diffuse>1 1 1 1</diffuse>
+          </material>
+      </visual>
+    </gazebo>
+    <gazebo reference="motor">
+      <visual>
+          <material>
+              <diffuse>1 1 1 1</diffuse>
+          </material>
+      </visual>
+    </gazebo>
+    <gazebo reference="palm_top_shell">
+      <visual>
+          <material>
+              <diffuse>1 1 1 1</diffuse>
+          </material>
+      </visual>
+    </gazebo>
+    <gazebo reference="right_finger_first_phalanx">
+      <visual>
+          <material>
+              <diffuse>1 1 1 1</diffuse>
+          </material>
+      </visual>
+    </gazebo>
+    <gazebo reference="right_external_rod">
+      <visual>
+          <material>
+              <diffuse>1 1 1 1</diffuse>
+          </material>
+      </visual>
+    </gazebo>
+    <gazebo reference="right_finger_last_phalanx">
+      <visual>
+          <material>
+              <diffuse>1 1 1 1</diffuse>
+          </material>
+      </visual>
+    </gazebo>
+    <gazebo reference="left_finger_first_phalanx">
+      <visual>
+          <material>
+              <diffuse>1 1 1 1</diffuse>
+          </material>
+      </visual>
+    </gazebo>
+    <gazebo reference="left_external_rod">
+      <visual>
+          <material>
+              <diffuse>1 1 1 1</diffuse>
+          </material>
+      </visual>
+    </gazebo>
+    <gazebo reference="left_finger_last_phalanx">
+      <visual>
+          <material>
+              <diffuse>1 1 1 1</diffuse>
+          </material>
+      </visual>
+    </gazebo>
   </xacro:macro>
 </robot>

File: gripper_pincette/description/ros2_control/gripper_pincette.ros2_control.xacro (robot description, xacro)
@@ -4,52 +4,52 @@
   <ros2_control name="${name}" type="system">
     <hardware>
-      <plugin>gazebo_ros2_control/GazeboSystem</plugin>
+      <plugin>ign_ros2_control/IgnitionSystem</plugin>
     </hardware>
-    <joint name="right_finger_joint">
-      <command_interface name="position"/>
-      <state_interface name="position"/>
-      <state_interface name="velocity"/>
-      <state_interface name="effort"/>
-    </joint>
-    <joint name="right_external_rod_joint">
-      <param name="mimic">right_finger_joint</param>
-      <param name="multiplier">-1</param>
-      <command_interface name="position"/>
-      <state_interface name="position"/>
-      <state_interface name="velocity"/>
-      <state_interface name="effort"/>
-    </joint>
-    <joint name="right_fingertip_joint">
-      <param name="mimic">right_finger_joint</param>
-      <param name="multiplier">-1</param>
-      <command_interface name="position"/>
-      <state_interface name="position"/>
-      <state_interface name="velocity"/>
-      <state_interface name="effort"/>
-    </joint>
-    <joint name="left_finger_joint">
-      <param name="mimic">right_finger_joint</param>
-      <param name="multiplier">-1</param>
-      <command_interface name="position"/>
-      <state_interface name="position"/>
-      <state_interface name="velocity"/>
-      <state_interface name="effort"/>
-    </joint>
-    <joint name="left_external_rod_joint">
-      <param name="mimic">right_finger_joint</param>
-      <param name="multiplier">-1</param>
-      <command_interface name="position"/>
-      <state_interface name="position"/>
-      <state_interface name="velocity"/>
-      <state_interface name="effort"/>
-    </joint>
-    <joint name="left_fingertip_joint">
-      <param name="mimic">right_finger_joint</param>
-      <param name="multiplier">-1</param>
-      <command_interface name="position"/>
-      <state_interface name="position"/>
-      <state_interface name="velocity"/>
-      <state_interface name="effort"/>
-    </joint>
+      <joint name="right_finger_joint">
+        <command_interface name="position"/>
+        <state_interface name="position"/>
+        <state_interface name="velocity"/>
+        <state_interface name="effort"/>
+      </joint>
+      <joint name="right_external_rod_joint">
+        <param name="mimic">right_finger_joint</param>
+        <param name="multiplier">-1</param>
+        <command_interface name="position"/>
+        <state_interface name="position"/>
+        <state_interface name="velocity"/>
+        <state_interface name="effort"/>
+      </joint>
+      <joint name="right_fingertip_joint">
+        <param name="mimic">right_finger_joint</param>
+        <param name="multiplier">-1</param>
+        <command_interface name="position"/>
+        <state_interface name="position"/>
+        <state_interface name="velocity"/>
+        <state_interface name="effort"/>
+      </joint>
+      <joint name="left_finger_joint">
+        <param name="mimic">right_finger_joint</param>
+        <param name="multiplier">-1</param>
+        <command_interface name="position"/>
+        <state_interface name="position"/>
+        <state_interface name="velocity"/>
+        <state_interface name="effort"/>
+      </joint>
+      <joint name="left_external_rod_joint">
+        <param name="mimic">right_finger_joint</param>
+        <param name="multiplier">-1</param>
+        <command_interface name="position"/>
+        <state_interface name="position"/>
+        <state_interface name="velocity"/>
+        <state_interface name="effort"/>
+      </joint>
+      <joint name="left_fingertip_joint">
+        <param name="mimic">right_finger_joint</param>
+        <param name="multiplier">-1</param>
+        <command_interface name="position"/>
+        <state_interface name="position"/>
+        <state_interface name="velocity"/>
+        <state_interface name="effort"/>
+      </joint>
   </ros2_control>
   </xacro:macro>

Commit message: (feat): add camera on explorer's gripper

File: explorer/description/gazebo/explorer.gazebo.xacro (robot description, xacro)
@@ -113,4 +113,25 @@
       </visual>
     </gazebo>
+    <gazebo reference="camera_explorer">
+      <sensor name="camera" type="camera">
+        <camera>
+          <optical_frame_id>camera_explorer</optical_frame_id>
+          <horizontal_fov>1.047</horizontal_fov>
+          <image>
+              <width>640</width>
+              <height>400</height>
+          </image>
+          <clip>
+              <near>0.05</near>
+              <far>100</far>
+          </clip>
+        </camera>
+        <always_on>1</always_on>
+        <update_rate>30</update_rate>
+        <visualize>true</visualize>
+        <topic>camera</topic>
+        <enable_metrics>false</enable_metrics>
+      </sensor>
+    </gazebo>
   </xacro:macro>
 </robot>

File: explorer/description/urdf/explorer.urdf.xacro (robot description, xacro)
@@ -8,4 +8,5 @@
   <!-- create link fixed to the "world" -->
   <link name="world"/>
+  <link name="camera_explorer"/>
   <!-- base_joint fixes base_link to the environment -->
   <joint name="base_joint" type="fixed">
@@ -26,4 +27,9 @@
     <child link="ft_frame"/>
     <origin xyz="0.011 0 0.15" rpy="0 0 0"/>
+  </joint>
+  <joint name="camera_joint" type="fixed">
+    <parent link="structure"/>
+    <child link="camera_explorer"/>
+    <origin xyz="0.011 0 0.105" rpy="0 ${-pi/2} 0"/>
   </joint>
   <joint name="joint-tool" type="fixed">
