Commit message: (feat): add gripper pincette

File: explorer/description/ros2_control/explorer.ros2_control.xacro (robot description, xacro)
@@ -95,4 +95,44 @@
         <state_interface name="velocity"/>
       </joint>
+      <joint name="right_finger_joint">
+        <command_interface name="position"/>
+        <state_interface name="position"/>
+        <state_interface name="velocity"/>
+      </joint>
+      <joint name="right_external_rod_joint">
+        <param name="mimic">right_finger_joint</param>
+        <param name="multiplier">-1</param>
+        <command_interface name="position"/>
+        <state_interface name="position"/>
+        <state_interface name="velocity"/>
+      </joint>
+      <joint name="right_fingertip_joint">
+        <param name="mimic">right_finger_joint</param>
+        <param name="multiplier">-1</param>
+        <command_interface name="position"/>
+        <state_interface name="position"/>
+        <state_interface name="velocity"/>
+      </joint>
+      <joint name="left_finger_joint">
+        <param name="mimic">right_finger_joint</param>
+        <param name="multiplier">-1</param>
+        <command_interface name="position"/>
+        <state_interface name="position"/>
+        <state_interface name="velocity"/>
+      </joint>
+      <joint name="left_external_rod_joint">
+        <param name="mimic">right_finger_joint</param>
+        <param name="multiplier">-1</param>
+        <command_interface name="position"/>
+        <state_interface name="position"/>
+        <state_interface name="velocity"/>
+      </joint>
+      <joint name="left_fingertip_joint">
+        <param name="mimic">right_finger_joint</param>
+        <param name="multiplier">-1</param>
+        <command_interface name="position"/>
+        <state_interface name="position"/>
+        <state_interface name="velocity"/>
+      </joint>
     </ros2_control>
   </xacro:macro>

File: explorer/description/urdf/explorer.urdf.xacro (robot description, xacro)
@@ -4,4 +4,5 @@
   <!-- Import explorer macro -->
   <xacro:include filename="$(find ros2_control_explorer)/description/urdf/explorer_old_description.urdf.xacro"/>
+  <xacro:include filename="$(find gripper_pincette)/description/urdf/gripper_pincette_description.urdf.xacro"/>
   <!-- create link fixed to the "world" -->
   <link name="world"/>
@@ -13,5 +14,23 @@
     <axis xyz="0 0 1"/>
   </joint>
+  <joint name="joint_6" type="revolute">
+    <parent link="link_5"/>
+    <child link="structure"/>
+    <origin xyz="0 0.090 0.083" rpy="${-(65*pi)/180} 0 0"/>
+    <axis xyz="0 0 1"/>
+    <limit effort="1000.0" lower="${-pi}" upper="${pi}" velocity="2.5"/>
+  </joint>
+  <joint name="joint-ft_frame" type="fixed">
+    <parent link="structure"/>
+    <child link="ft_frame"/>
+    <origin xyz="0.011 0 0.15" rpy="0 0 0"/>
+  </joint>
+  <joint name="joint-tool" type="fixed">
+    <parent link="ft_frame"/>
+    <child link="tool0"/>
+    <origin xyz="0 0 0" rpy="0 0 0"/>
+  </joint>
   <xacro:explorer_old_description/>
+  <xacro:gripper_pincette/>
   <!-- Import explorer ros2_control description -->
   <xacro:include filename="$(find ros2_control_explorer)/description/ros2_control/explorer.ros2_control.xacro" />

File: explorer/description/urdf/explorer_old_description.urdf.xacro (robot description, xacro)
@@ -94,5 +94,5 @@
       izz="0.00092964379"
   />
-  <xacro:create_link
+  <!-- <xacro:create_link
       link_name="link_6"
       xyz_offset="0 0 0"
@@ -108,5 +108,5 @@
       iyz="2.73718e-7"
       izz="0.000713799995"
-  />
+  /> -->
   <link name="ft_frame"/>
   <link name="tool0"/>
@@ -147,4 +147,5 @@
     <limit effort="1000.0" lower="${-pi}" upper="${pi}" velocity="2.5"/>
   </joint>
+<!--
   <joint name="joint_6" type="revolute">
     <parent link="link_5"/>
@@ -163,5 +164,5 @@
     <child link="tool0"/>
     <origin xyz="0 0 0" rpy="0 0 0"/>
-  </joint>
+  </joint> -->
 </xacro:macro>
 </robot>

Commit message: (fix): change max velocity

File: explorer/description/ros2_control/explorer.ros2_control.xacro (robot description, xacro)
@@ -17,6 +17,6 @@
         </command_interface>
         <command_interface name="velocity">
-          <param name="min">-2.5</param>
-          <param name="max">2.5</param>
+          <param name="min">-0.5</param>
+          <param name="max">0.5</param>
         </command_interface>
         <state_interface name="position">
@@ -31,6 +31,6 @@
         </command_interface>
         <command_interface name="velocity">
-          <param name="min">-2.5</param>
-          <param name="max">2.5</param>
+          <param name="min">-0.5</param>
+          <param name="max">0.5</param>
         </command_interface>
         <state_interface name="position">
@@ -45,6 +45,6 @@
         </command_interface>
         <command_interface name="velocity">
-          <param name="min">-2.5</param>
-          <param name="max">2.5</param>
+          <param name="min">-0.5</param>
+          <param name="max">0.5</param>
         </command_interface>
         <state_interface name="position">
@@ -59,6 +59,6 @@
         </command_interface>
         <command_interface name="velocity">
-          <param name="min">-2.5</param>
-          <param name="max">2.5</param>
+          <param name="min">-0.5</param>
+          <param name="max">0.5</param>
         </command_interface>
         <state_interface name="position">
@@ -73,6 +73,6 @@
         </command_interface>
         <command_interface name="velocity">
-          <param name="min">-2.5</param>
-          <param name="max">2.5</param>
+          <param name="min">-0.5</param>
+          <param name="max">0.5</param>
         </command_interface>
         <state_interface name="position">
@@ -87,6 +87,6 @@
         </command_interface>
         <command_interface name="velocity">
-          <param name="min">-2.5</param>
-          <param name="max">2.5</param>
+          <param name="min">-0.5</param>
+          <param name="max">0.5</param>
         </command_interface>
         <state_interface name="position">

File: explorer/description/urdf/explorer_old_description.urdf.xacro (robot description, xacro)
@@ -117,5 +117,5 @@
     <origin xyz="0 0 0.0555" rpy="0 0 0"/>
     <axis xyz="0 0 1"/>
-    <limit effort="1000.0" lower="${-pi}" upper="${pi}" velocity="2.5"/>
+    <limit effort="1000.0" lower="${-pi}" upper="${pi}" velocity="0.5"/>
   </joint>
   <joint name="joint_2" type="revolute">
@@ -124,5 +124,5 @@
     <origin xyz="0 0.0245 0.058952" rpy="${pi/2} ${-pi/2} 0"/>
     <axis xyz="0 0 1"/>
-    <limit effort="1000.0" lower="${-pi/2}" upper="${pi/2}" velocity="2.5"/>
+    <limit effort="1000.0" lower="${-pi/2}" upper="${pi/2}" velocity="0.5"/>
   </joint>
   <joint name="joint_3" type="revolute">
@@ -131,5 +131,5 @@
     <origin xyz="0.409872 0 -0.002" rpy="${pi} 0 ${-pi/2}"/>
     <axis xyz="0 0 1"/>
-    <limit effort="1000.0" lower="${-3*pi/2}" upper="${pi/2}" velocity="2.5"/>
+    <limit effort="1000.0" lower="${-3*pi/2}" upper="${pi/2}" velocity="0.5"/>
   </joint>
   <joint name="joint_4" type="revolute">
@@ -138,5 +138,5 @@
     <origin xyz="0.2339 0 -0.014" rpy="0 ${pi/2} 0"/>
     <axis xyz="0 0 1"/>
-    <limit effort="1000.0" lower="${-pi}" upper="${pi}" velocity="2.5"/>
+    <limit effort="1000.0" lower="${-pi}" upper="${pi}" velocity="0.5"/>
   </joint>
   <joint name="joint_5" type="revolute">
@@ -145,5 +145,5 @@
     <origin xyz="0 0.090 0.083" rpy="${(65*pi)/180} 0 ${pi}"/>
     <axis xyz="0 0 1"/>
-    <limit effort="1000.0" lower="${-pi}" upper="${pi}" velocity="2.5"/>
+    <limit effort="1000.0" lower="${-pi}" upper="${pi}" velocity="0.5"/>
   </joint>
 <!--
@@ -153,5 +153,5 @@
     <origin xyz="0 0.090 0.083" rpy="${-(65*pi)/180} 0 0"/>
     <axis xyz="0 0 1"/>
-    <limit effort="1000.0" lower="${-pi}" upper="${pi}" velocity="2.5"/>
+    <limit effort="1000.0" lower="${-pi}" upper="${pi}" velocity="0.5"/>
   </joint>
   <joint name="joint-ft_frame" type="fixed">

Commit message: feat: add Actuator HW interfaces, explorer communication bridge (and simulator)

File: explorer/description/ros2_control/explorer.ros2_control.xacro (robot description, xacro)
@@ -2,4 +2,5 @@
 <robot xmlns:xacro="http://www.ros.org/wiki/xacro">
   <xacro:macro name="explorer_ros2_control" params="name use_ignition:=^|false">
+    <xacro:include filename="$(find ros2_control_explorer)/description/urdf/explorer_joints.xacro" />
     <ros2_control name="${name}" type="system">
       <hardware>
@@ -11,134 +12,11 @@
         </xacro:unless>
       </hardware>
-      <joint name="joint_1">
-        <command_interface name="position">
-          <param name="min">{-pi}</param>
-          <param name="max">{pi}</param>
-        </command_interface>
-        <command_interface name="velocity">
-          <param name="min">-0.5</param>
-          <param name="max">0.5</param>
-        </command_interface>
-        <state_interface name="position">
-          <param name="initial_value">0.0</param>
-        </state_interface>
-        <state_interface name="velocity"/>
-      </joint>
-      <joint name="joint_2">
-        <command_interface name="position">
-          <param name="min">{-pi/2}</param>
-          <param name="max">{pi/2}</param>
-        </command_interface>
-        <command_interface name="velocity">
-          <param name="min">-0.5</param>
-          <param name="max">0.5</param>
-        </command_interface>
-        <state_interface name="position">
-          <param name="initial_value">0.0</param>
-        </state_interface>
-        <state_interface name="velocity"/>
-      </joint>
-      <joint name="joint_3">
-        <command_interface name="position">
-          <param name="min">{-3*pi/2}</param>
-          <param name="max">{pi/2}</param>
-        </command_interface>
-        <command_interface name="velocity">
-          <param name="min">-0.5</param>
-          <param name="max">0.5</param>
-        </command_interface>
-        <state_interface name="position">
-          <param name="initial_value">0.0</param>
-        </state_interface>
-        <state_interface name="velocity"/>
-      </joint>
-      <joint name="joint_4">
-        <command_interface name="position">
-          <param name="min">{-pi}</param>
-          <param name="max">{pi}</param>
-        </command_interface>
-        <command_interface name="velocity">
-          <param name="min">-0.5</param>
-          <param name="max">0.5</param>
-        </command_interface>
-        <state_interface name="position">
-          <param name="initial_value">0.0</param>
-        </state_interface>
-        <state_interface name="velocity"/>
-      </joint>
-      <joint name="joint_5">
-        <command_interface name="position">
-          <param name="min">{-pi}</param>
-          <param name="max">{pi}</param>
-        </command_interface>
-        <command_interface name="velocity">
-          <param name="min">-0.5</param>
-          <param name="max">0.5</param>
-        </command_interface>
-        <state_interface name="position">
-          <param name="initial_value">0.0</param>
-        </state_interface>
-        <state_interface name="velocity"/>
-      </joint>
-      <joint name="joint_6">
-        <command_interface name="position">
-          <param name="min">{-pi}</param>
-          <param name="max">{pi}</param>
-        </command_interface>
-        <command_interface name="velocity">
-          <param name="min">-0.5</param>
-          <param name="max">0.5</param>
-        </command_interface>
-        <state_interface name="position">
-          <param name="initial_value">0.0</param>
-        </state_interface>
-        <state_interface name="velocity"/>
-      </joint>
-      <joint name="right_finger_joint">
-        <command_interface name="position"/>
-        <state_interface name="position"/>
-        <state_interface name="velocity"/>
-        <state_interface name="effort"/>
-      </joint>
-      <joint name="right_external_rod_joint">
-        <param name="mimic">right_finger_joint</param>
-        <param name="multiplier">-1</param>
-        <command_interface name="position"/>
-        <state_interface name="position"/>
-        <state_interface name="velocity"/>
-        <state_interface name="effort"/>
-      </joint>
-      <joint name="right_fingertip_joint">
-        <param name="mimic">right_finger_joint</param>
-        <param name="multiplier">-1</param>
-        <command_interface name="position"/>
-        <state_interface name="position"/>
-        <state_interface name="velocity"/>
-        <state_interface name="effort"/>
-      </joint>
-      <joint name="left_finger_joint">
-        <param name="mimic">right_finger_joint</param>
-        <param name="multiplier">-1</param>
-        <command_interface name="position"/>
-        <state_interface name="position"/>
-        <state_interface name="velocity"/>
-        <state_interface name="effort"/>
-      </joint>
-      <joint name="left_external_rod_joint">
-        <param name="mimic">right_finger_joint</param>
-        <param name="multiplier">-1</param>
-        <command_interface name="position"/>
-        <state_interface name="position"/>
-        <state_interface name="velocity"/>
-        <state_interface name="effort"/>
-      </joint>
-      <joint name="left_fingertip_joint">
-        <param name="mimic">right_finger_joint</param>
-        <param name="multiplier">-1</param>
-        <command_interface name="position"/>
-        <state_interface name="position"/>
-        <state_interface name="velocity"/>
-        <state_interface name="effort"/>
-      </joint>
+      <xacro:explorer_joint_1 />
+      <xacro:explorer_joint_2 />
+      <xacro:explorer_joint_3 />
+      <xacro:explorer_joint_4 />
+      <xacro:explorer_joint_5 />
+      <xacro:explorer_joint_6 />
+      <xacro:explorer_gripper_joints />
     </ros2_control>
   </xacro:macro>

File: explorer/description/urdf/explorer.urdf.xacro (robot description, xacro)
@@ -2,4 +2,5 @@
 <robot xmlns:xacro="http://wiki.ros.org/xacro" name="explorer">
   <xacro:arg name="use_ignition" default="false" />
+  <xacro:arg name="use_actuator_interface" default="false" />
   <!-- Import explorer macro -->
   <xacro:include filename="$(find ros2_control_explorer)/description/urdf/explorer_old_description.urdf.xacro"/>
@@ -34,6 +35,12 @@
   <xacro:gripper_pincette/>
   <!-- Import explorer ros2_control description -->
-  <xacro:include filename="$(find ros2_control_explorer)/description/ros2_control/explorer.ros2_control.xacro" />
-  <xacro:explorer_ros2_control name="explorer" use_ignition="$(arg use_ignition)"/>
+  <xacro:unless value="$(arg use_actuator_interface)">
+    <xacro:include filename="$(find ros2_control_explorer)/description/ros2_control/explorer.ros2_control.xacro" />
+    <xacro:explorer_ros2_control name="explorer" use_ignition="$(arg use_ignition)"/>
+  </xacro:unless>
+  <xacro:if value="$(arg use_actuator_interface)">
+    <xacro:include filename="$(find ros2_control_explorer)/description/ros2_control/explorer_actuators.ros2_control.xacro" />
+    <xacro:explorer_ros2_control name="explorer" use_ignition="$(arg use_ignition)" />
+  </xacro:if>
   <xacro:if value="$(arg use_ignition)">
     <!-- Import Gazebo definitions + plugin -->

Commit message: PoC to support servo joint for gripper

File: explorer/description/ros2_control/explorer.ros2_control.xacro (robot description, xacro)
@@ -18,4 +18,5 @@
       <xacro:explorer_joint_5 />
       <xacro:explorer_joint_6 />
+      <xacro:explorer_gripper_servo_joint />
       <xacro:explorer_gripper_joints />
     </ros2_control>

File: explorer/description/ros2_control/explorer_actuators.ros2_control.xacro (robot description, xacro)
@@ -40,4 +40,5 @@
     </hardware>
     <xacro:explorer_joint_6 />
+    <xacro:explorer_gripper_servo_joint />
   </ros2_control>
   <ros2_control name="${name}_gripper" type="system">

File: explorer/description/urdf/explorer_joints.xacro (robot description, xacro)
@@ -97,10 +97,21 @@
       </joint>
     </xacro:macro>
-    <xacro:macro name="explorer_gripper_joints">
+    <xacro:macro name="explorer_gripper_servo_joint">
       <joint name="right_finger_joint">
-        <command_interface name="position"/>
-        <state_interface name="position"/>
+        <command_interface name="position">
+          <param name="min">{-2*pi}</param>
+          <param name="max">{2*pi}</param>
+        </command_interface>
+        <command_interface name="velocity">
+          <param name="min">-3.2</param>
+          <param name="max">3.2</param>
+        </command_interface>
+        <state_interface name="position">
+          <param name="initial_value">0.0</param>
+        </state_interface>
         <state_interface name="velocity"/>
       </joint>
+    </xacro:macro>
+    <xacro:macro name="explorer_gripper_joints">
       <joint name="right_external_rod_joint">
         <param name="mimic">right_finger_joint</param>

Commit message: Dirty PoC replacing PyVESC with VESCpp

File: explorer/description/ros2_control/explorer.ros2_control.xacro (robot description, xacro)
@@ -1,5 +1,5 @@
 <?xml version="1.0"?>
 <robot xmlns:xacro="http://www.ros.org/wiki/xacro">
-  <xacro:macro name="explorer_ros2_control" params="name use_ignition:=^|false">
+  <xacro:macro name="explorer_ros2_control" params="name use_ignition:=^|false can_port:=^|vxcan1 host_id:=^|45">
     <xacro:include filename="$(find ros2_control_explorer)/description/urdf/explorer_joints.xacro" />
     <ros2_control name="${name}" type="system">

File: explorer/description/ros2_control/explorer_actuators.ros2_control.xacro (robot description, xacro)
@@ -2,9 +2,11 @@
 <robot xmlns:xacro="http://www.ros.org/wiki/xacro">
   <xacro:include filename="$(find ros2_control_explorer)/description/urdf/explorer_joints.xacro" />
-  <xacro:macro name="explorer_ros2_control" params="name use_ignition:=^|false">
+  <xacro:macro name="explorer_ros2_control" params="name use_ignition:=^|false can_port:=^|vxcan1  host_id:=^|45">
   <!-- ROS2 Control -->
   <ros2_control name="${name}_joint_1" type="actuator">
     <hardware>
       <plugin>orthopus_vesc_interface/VESCInterface</plugin>
+      <param name="host_id">${host_id}</param>
+      <param name="can_port">${can_port}</param>
       <param name="can_id">11</param>
     </hardware>
@@ -14,4 +16,6 @@
     <hardware>
       <plugin>orthopus_vesc_interface/VESCInterface</plugin>
+      <param name="host_id">${host_id}</param>
+      <param name="can_port">${can_port}</param>
       <param name="can_id">12</param>
     </hardware>
@@ -21,4 +25,6 @@
     <hardware>
       <plugin>orthopus_vesc_interface/VESCInterface</plugin>
+      <param name="host_id">${host_id}</param>
+      <param name="can_port">${can_port}</param>
       <param name="can_id">13</param>
     </hardware>
@@ -28,4 +34,6 @@
     <hardware>
       <plugin>orthopus_vesc_interface/VESCInterface</plugin>
+      <param name="host_id">${host_id}</param>
+      <param name="can_port">${can_port}</param>
       <param name="can_id">14</param>
     </hardware>
@@ -35,4 +43,6 @@
     <hardware>
       <plugin>orthopus_vesc_interface/VESCInterface</plugin>
+      <param name="host_id">${host_id}</param>
+      <param name="can_port">${can_port}</param>
       <param name="can_id">15</param>
     </hardware>
@@ -42,4 +52,6 @@
     <hardware>
       <plugin>orthopus_vesc_interface/VESCInterface</plugin>
+      <param name="host_id">${host_id}</param>
+      <param name="can_port">${can_port}</param>
       <param name="can_id">16</param>
     </hardware>

File: explorer/description/urdf/explorer.urdf.xacro (robot description, xacro)
@@ -3,4 +3,6 @@
   <xacro:arg name="use_ignition" default="false" />
   <xacro:arg name="use_actuator_interface" default="false" />
+  <xacro:arg name="can_port" default="vxcan1" />
+  <xacro:arg name="host_id" default="45" />
   <xacro:arg name="use_POC2" default="false" />
   <xacro:include filename="$(find gripper_pincette)/description/urdf/gripper_pincette_description.urdf.xacro"/>
@@ -58,9 +60,9 @@
   <xacro:unless value="$(arg use_actuator_interface)">
     <xacro:include filename="$(find ros2_control_explorer)/description/ros2_control/explorer.ros2_control.xacro" />
-    <xacro:explorer_ros2_control name="explorer" use_ignition="$(arg use_ignition)"/>
+    <xacro:explorer_ros2_control name="explorer" use_ignition="$(arg use_ignition)" can_port="$(arg can_port)"  host_id="$(arg host_id)" />
   </xacro:unless>
   <xacro:if value="$(arg use_actuator_interface)">
     <xacro:include filename="$(find ros2_control_explorer)/description/ros2_control/explorer_actuators.ros2_control.xacro" />
-    <xacro:explorer_ros2_control name="explorer" use_ignition="$(arg use_ignition)" />
+    <xacro:explorer_ros2_control name="explorer" use_ignition="$(arg use_ignition)" can_port="$(arg can_port)"  host_id="$(arg host_id)" />
   </xacro:if>
   <xacro:if value="$(arg use_ignition)">

File: explorer/description/urdf/explorer_joints.xacro (robot description, xacro)
@@ -103,12 +103,12 @@
           <param name="max">{2*pi}</param>
         </command_interface>
-        <command_interface name="velocity">
+        <!--command_interface name="velocity">
           <param name="min">-0.5</param>
           <param name="max">0.5</param>
-        </command_interface>
+        </command_interface-->
         <state_interface name="position">
           <param name="initial_value">0.0</param>
         </state_interface>
-        <state_interface name="velocity"/>
+        <!--state_interface name="velocity"/-->
       </joint>
     </xacro:macro>
@@ -119,5 +119,5 @@
         <command_interface name="position"/>
         <state_interface name="position"/>
-        <state_interface name="velocity"/>
+        <!--state_interface name="velocity"/-->
       </joint>
       <joint name="right_fingertip_joint">
@@ -126,5 +126,5 @@
         <command_interface name="position"/>
         <state_interface name="position"/>
-        <state_interface name="velocity"/>
+        <!--state_interface name="velocity"/-->
       </joint>
       <joint name="left_finger_joint">
@@ -133,5 +133,5 @@
         <command_interface name="position"/>
         <state_interface name="position"/>
-        <state_interface name="velocity"/>
+        <!--state_interface name="velocity"/-->
       </joint>
       <joint name="left_external_rod_joint">
@@ -140,5 +140,5 @@
         <command_interface name="position"/>
         <state_interface name="position"/>
-        <state_interface name="velocity"/>
+        <!--state_interface name="velocity"/-->
       </joint>
       <joint name="left_fingertip_joint">
@@ -147,5 +147,5 @@
         <command_interface name="position"/>
         <state_interface name="position"/>
-        <state_interface name="velocity"/>
+        <!--state_interface name="velocity"/-->
       </joint>
     </xacro:macro>
