Commit message: feat: Add AUX streaming, add parameters, simply ros_control urdf stuff

File: explorer/description/ros2_control/explorer_actuators.ros2_control.xacro (robot description, xacro)
@@ -2,11 +2,16 @@
 <robot xmlns:xacro="http://www.ros.org/wiki/xacro">
   <xacro:include filename="$(find ros2_control_explorer)/description/urdf/explorer_joints.xacro" />
-  <xacro:macro name="explorer_ros2_control" params="name use_ignition:=^|false can_port:=^|vxcan1  host_id:=^|45">
+  <xacro:macro name="explorer_ros2_control" params="name use_ignition:=^|false can_port:=^|vxcan1  host_id:=^|45 rt_stream_rate:=^|250 aux_stream_rate:=^|10">
+    <xacro:macro name="hw_intf_params">
+      <plugin>orthopus_vesc_interface/VESCInterface</plugin>
+      <param name="host_id">${host_id}</param>
+      <param name="can_port">${can_port}</param>
+      <param name="rt_stream_rate">${rt_stream_rate}</param>
+      <param name="aux_stream_rate">${aux_stream_rate}</param>
+    </xacro:macro>
   <!-- ROS2 Control -->
   <ros2_control name="${name}_joint_1" type="actuator">
     <hardware>
-      <plugin>orthopus_vesc_interface/VESCInterface</plugin>
-      <param name="host_id">${host_id}</param>
-      <param name="can_port">${can_port}</param>
+       <xacro:hw_intf_params />
       <param name="can_id">11</param>
     </hardware>
@@ -15,7 +20,5 @@
   <ros2_control name="${name}_joint_2" type="actuator">
     <hardware>
-      <plugin>orthopus_vesc_interface/VESCInterface</plugin>
-      <param name="host_id">${host_id}</param>
-      <param name="can_port">${can_port}</param>
+       <xacro:hw_intf_params />
       <param name="can_id">12</param>
     </hardware>
@@ -24,7 +27,5 @@
   <ros2_control name="${name}_joint_3" type="actuator">
     <hardware>
-      <plugin>orthopus_vesc_interface/VESCInterface</plugin>
-      <param name="host_id">${host_id}</param>
-      <param name="can_port">${can_port}</param>
+       <xacro:hw_intf_params />
       <param name="can_id">13</param>
     </hardware>
@@ -33,7 +34,5 @@
   <ros2_control name="${name}_joint_4" type="actuator">
     <hardware>
-      <plugin>orthopus_vesc_interface/VESCInterface</plugin>
-      <param name="host_id">${host_id}</param>
-      <param name="can_port">${can_port}</param>
+       <xacro:hw_intf_params />
       <param name="can_id">14</param>
     </hardware>
@@ -42,7 +41,5 @@
   <ros2_control name="${name}_joint_5" type="actuator">
     <hardware>
-      <plugin>orthopus_vesc_interface/VESCInterface</plugin>
-      <param name="host_id">${host_id}</param>
-      <param name="can_port">${can_port}</param>
+       <xacro:hw_intf_params />
       <param name="can_id">15</param>
     </hardware>
@@ -51,7 +48,5 @@
   <ros2_control name="${name}_joint_6" type="actuator">
     <hardware>
-      <plugin>orthopus_vesc_interface/VESCInterface</plugin>
-      <param name="host_id">${host_id}</param>
-      <param name="can_port">${can_port}</param>
+       <xacro:hw_intf_params />
       <param name="can_id">16</param>
     </hardware>

File: explorer/description/urdf/explorer.urdf.xacro (robot description, xacro)
@@ -5,4 +5,6 @@
   <xacro:arg name="can_port" default="vxcan1" />
   <xacro:arg name="host_id" default="45" />
+  <xacro:arg name="rt_stream_rate" default="250" />
+  <xacro:arg name="aux_stream_rate" default="10" />
   <xacro:arg name="use_POC2" default="false" />
   <xacro:include filename="$(find gripper_pincette)/description/urdf/gripper_pincette_description.urdf.xacro"/>
@@ -60,9 +62,16 @@
   <xacro:unless value="$(arg use_actuator_interface)">
     <xacro:include filename="$(find ros2_control_explorer)/description/ros2_control/explorer.ros2_control.xacro" />
-    <xacro:explorer_ros2_control name="explorer" use_ignition="$(arg use_ignition)" can_port="$(arg can_port)"  host_id="$(arg host_id)" />
+    <xacro:explorer_ros2_control name="explorer" use_ignition="$(arg use_ignition)" />
   </xacro:unless>
   <xacro:if value="$(arg use_actuator_interface)">
     <xacro:include filename="$(find ros2_control_explorer)/description/ros2_control/explorer_actuators.ros2_control.xacro" />
-    <xacro:explorer_ros2_control name="explorer" use_ignition="$(arg use_ignition)" can_port="$(arg can_port)"  host_id="$(arg host_id)" />
+    <xacro:explorer_ros2_control
+      name="explorer"
+      use_ignition="$(arg use_ignition)"
+      can_port="$(arg can_port)"
+      host_id="$(arg host_id)"
+      rt_stream_rate="$(arg rt_stream_rate)"
+      aux_stream_rate="$(arg aux_stream_rate)"
+    />
   </xacro:if>
   <xacro:if value="$(arg use_ignition)">
