Commit message: (fix): reverse joint rotation direction on POC2

File: explorer/description/urdf/explorer_POC2_description.urdf.xacro (robot description, xacro)
@@ -116,5 +116,5 @@
     <child link="link_1"/>
     <origin xyz="0 0 0.0555" rpy="0 0 0"/>
-    <axis xyz="0 0 1"/>
+    <axis xyz="0 0 -1"/>
     <limit effort="1000.0" lower="${-pi}" upper="${pi}" velocity="2.5"/>
   </joint>
@@ -123,5 +123,5 @@
     <child link="link_2"/>
     <origin xyz="0 0.0265 0.058952" rpy="${pi/2} ${-pi/2} 0"/>
-    <axis xyz="0 0 1"/>
+    <axis xyz="0 0 -1"/>
     <limit effort="1000.0" lower="${-pi/2}" upper="${pi/2}" velocity="2.5"/>
   </joint>
@@ -130,5 +130,5 @@
     <child link="link_3"/>
     <origin xyz="0.413 0 0" rpy="${pi} 0 ${-pi/2}"/>
-    <axis xyz="0 0 1"/>
+    <axis xyz="0 0 -1"/>
     <limit effort="1000.0" lower="${-3*pi/2}" upper="${pi/2}" velocity="2.5"/>
   </joint>
@@ -137,5 +137,5 @@
     <child link="link_4"/>
     <origin xyz="0.1885 0 -0.008" rpy="${pi/2} 0 ${pi/2}"/>
-    <axis xyz="0 0 1"/>
+    <axis xyz="0 0 -1"/>
     <limit effort="1000.0" lower="${-pi}" upper="${pi}" velocity="2.5"/>
   </joint>
@@ -144,5 +144,5 @@
     <child link="link_5"/>
     <origin xyz="0 0.0285 0.1" rpy="${pi/2} 0 ${pi}"/>
-    <axis xyz="0 0 1"/>
+    <axis xyz="0 0 -1"/>
     <limit effort="1000.0" lower="${-pi}" upper="${pi}" velocity="2.5"/>
   </joint>

Commit message: (fix) : change pos 0 POC2

File: explorer/description/urdf/explorer_POC2_description.urdf.xacro (robot description, xacro)
@@ -129,5 +129,5 @@
     <parent link="link_2"/>
     <child link="link_3"/>
-    <origin xyz="0.413 0 0" rpy="${pi} 0 ${-pi/2}"/>
+    <origin xyz="0.413 0 0" rpy="${pi} 0 0"/>
     <axis xyz="0 0 -1"/>
     <limit effort="1000.0" lower="${-3*pi/2}" upper="${pi/2}" velocity="2.5"/>

Commit message: (fix) : fix POC2 limits

File: explorer/description/urdf/explorer_POC2_description.urdf.xacro (robot description, xacro)
@@ -117,5 +117,5 @@
     <origin xyz="0 0 0.0555" rpy="0 0 0"/>
     <axis xyz="0 0 -1"/>
-    <limit effort="1000.0" lower="${-pi}" upper="${pi}" velocity="10"/>
+    <limit effort="1000.0" lower="-2.97" upper="2.97" velocity="10"/>
   </joint>
   <joint name="joint_2" type="revolute">
@@ -124,5 +124,5 @@
     <origin xyz="0 0.0265 0.058952" rpy="${pi/2} ${-pi/2} 0"/>
     <axis xyz="0 0 -1"/>
-    <limit effort="1000.0" lower="${-pi/2}" upper="${pi/2}" velocity="10"/>
+    <limit effort="1000.0" lower="-2.14" upper="2.14" velocity="10"/>
   </joint>
   <joint name="joint_3" type="revolute">
@@ -131,5 +131,5 @@
     <origin xyz="0.413 0 0" rpy="${pi} 0 0"/>
     <axis xyz="0 0 -1"/>
-    <limit effort="1000.0" lower="${-3*pi/2}" upper="${pi/2}" velocity="10"/>
+    <limit effort="1000.0" lower="-2.97" upper="2.97" velocity="10"/>
   </joint>
   <joint name="joint_4" type="revolute">
@@ -138,5 +138,5 @@
     <origin xyz="0.1885 0 -0.008" rpy="${pi/2} ${pi} ${pi/2}"/>
     <axis xyz="0 0 -1"/>
-    <limit effort="1000.0" lower="${-pi}" upper="${pi}" velocity="10"/>
+    <limit effort="1000.0" lower="-2.97" upper="2.97" velocity="10"/>
   </joint>
   <joint name="joint_5" type="revolute">
@@ -145,5 +145,5 @@
     <origin xyz="0 0.0285 0.1" rpy="${pi/2} 0 ${pi}"/>
     <axis xyz="0 0 -1"/>
-    <limit effort="1000.0" lower="${-pi}" upper="${pi}" velocity="10"/>
+    <limit effort="1000.0" lower="-1.8" upper="1.8" velocity="10"/>
   </joint>
   <!-- <joint name="joint_6" type="revolute">
