Commit message: (fix): fix explorer urdf to work with and without wheelchair

File: explorer/description/urdf/explorer.urdf.xacro (robot description, xacro)
@@ -5,5 +5,12 @@
   <xacro:include filename="$(find ros2_control_explorer)/description/urdf/explorer_old_description.urdf.xacro"/>
   <!-- create link fixed to the "world" -->
-  <!-- <link name="world"/> -->
+  <link name="world"/>
+  <!-- base_joint fixes base_link to the environment -->
+  <joint name="base_joint" type="fixed">
+    <parent link="world"/>
+    <child link="base_link"/>
+    <origin xyz="0 0 0" rpy="0 0 0"/>
+    <axis xyz="0 0 1"/>
+  </joint>
   <xacro:explorer_old_description/>
   <!-- Import explorer ros2_control description -->

File: explorer/description/urdf/explorer_new_description.urdf.xacro (robot description, xacro)
@@ -111,11 +111,4 @@
   <link name="ft_frame"/>
   <link name="tool0"/>
-  <!-- base_joint fixes base_link to the environment -->
-  <joint name="base_joint" type="fixed">
-    <parent link="world"/>
-    <child link="base_link"/>
-    <origin xyz="0 0 0" rpy="0 0 0"/>
-    <axis xyz="0 0 1"/>
-  </joint>
   <!-- joints - main serial chain -->
   <joint name="joint_1" type="revolute">

File: explorer/description/urdf/explorer_old_description.urdf.xacro (robot description, xacro)
@@ -111,11 +111,4 @@
   <link name="ft_frame"/>
   <link name="tool0"/>
-  <!-- base_joint fixes base_link to the environment -->
-  <!-- <joint name="base_joint" type="fixed">
-    <parent link="world"/>
-    <child link="base_link"/>
-    <origin xyz="0 0 0" rpy="0 0 0"/>
-    <axis xyz="0 0 1"/>
-  </joint> -->
   <!-- joints - main serial chain -->
   <joint name="joint_1" type="revolute">

Commit message: (fix): fix urdf files to get a proper default position

File: explorer/description/urdf/explorer.urdf.xacro (robot description, xacro)
@@ -18,5 +18,5 @@
     <parent link="link_5"/>
     <child link="structure"/>
-    <origin xyz="0 0.090 0.083" rpy="${-(65*pi)/180} 0 0"/>
+    <origin xyz="0 0.090 0.083" rpy="0 ${(65*pi)/180} ${pi/2}"/>
     <axis xyz="0 0 1"/>
     <limit effort="1000.0" lower="${-pi}" upper="${pi}" velocity="2.5"/>

File: explorer/description/urdf/explorer_old_description.urdf.xacro (robot description, xacro)
@@ -136,5 +136,5 @@
     <parent link="link_3"/>
     <child link="link_4"/>
-    <origin xyz="0.2339 0 -0.014" rpy="0 ${pi/2} 0"/>
+    <origin xyz="0.2339 0 -0.014" rpy="0 ${3*pi/2} ${pi}"/>
     <axis xyz="0 0 1"/>
     <limit effort="1000.0" lower="${-pi}" upper="${pi}" velocity="0.5"/>

Commit message: First cartesian working demo

File: explorer/description/urdf/explorer.urdf.xacro (robot description, xacro)
@@ -20,5 +20,5 @@
     <child link="structure"/>
     <origin xyz="0 0.090 0.083" rpy="0 ${(65*pi)/180} ${pi/2}"/>
-    <axis xyz="0 0 1"/>
+    <axis xyz="0 0 -1"/>
     <limit effort="1000.0" lower="${-pi}" upper="${pi}" velocity="2.5"/>
   </joint>

File: explorer/description/urdf/explorer_old_description.urdf.xacro (robot description, xacro)
@@ -116,5 +116,5 @@
     <child link="link_1"/>
     <origin xyz="0 0 0.0555" rpy="0 0 0"/>
-    <axis xyz="0 0 1"/>
+    <axis xyz="0 0 -1"/>
     <limit effort="1000.0" lower="${-pi}" upper="${pi}" velocity="0.5"/>
   </joint>
@@ -123,6 +123,6 @@
     <child link="link_2"/>
     <origin xyz="0 0.0245 0.058952" rpy="${pi/2} ${-pi/2} 0"/>
-    <axis xyz="0 0 1"/>
-    <limit effort="1000.0" lower="${-pi/2}" upper="${pi/2}" velocity="0.5"/>
+    <axis xyz="0 0 -1"/>
+    <limit effort="1000.0" lower="${-pi}" upper="${pi}" velocity="0.5"/>
   </joint>
   <joint name="joint_3" type="revolute">
@@ -130,5 +130,5 @@
     <child link="link_3"/>
     <origin xyz="0.409872 0 -0.002" rpy="${pi} 0 ${-pi/2}"/>
-    <axis xyz="0 0 1"/>
+    <axis xyz="0 0 -1"/>
     <limit effort="1000.0" lower="${-3*pi/2}" upper="${pi/2}" velocity="0.5"/>
   </joint>
@@ -137,5 +137,5 @@
     <child link="link_4"/>
     <origin xyz="0.2339 0 -0.014" rpy="0 ${3*pi/2} ${pi}"/>
-    <axis xyz="0 0 1"/>
+    <axis xyz="0 0 -1"/>
     <limit effort="1000.0" lower="${-pi}" upper="${pi}" velocity="0.5"/>
   </joint>
@@ -144,5 +144,5 @@
     <child link="link_5"/>
     <origin xyz="0 0.090 0.083" rpy="${(65*pi)/180} 0 ${pi}"/>
-    <axis xyz="0 0 1"/>
+    <axis xyz="0 0 -1"/>
     <limit effort="1000.0" lower="${-pi}" upper="${pi}" velocity="0.5"/>
   </joint>

Commit message: (fix): fix gazebo simulation

File: explorer/description/urdf/explorer.urdf.xacro (robot description, xacro)
@@ -21,5 +21,5 @@
     <origin xyz="0 0.090 0.083" rpy="0 ${(65*pi)/180} ${pi/2}"/>
     <axis xyz="0 0 -1"/>
-    <limit effort="1000.0" lower="${-pi}" upper="${pi}" velocity="2.5"/>
+    <limit effort="1000.0" lower="${-pi}" upper="${pi}" velocity="10"/>
   </joint>
   <joint name="joint-ft_frame" type="fixed">

File: explorer/description/urdf/explorer_old_description.urdf.xacro (robot description, xacro)
@@ -117,5 +117,5 @@
     <origin xyz="0 0 0.0555" rpy="0 0 0"/>
     <axis xyz="0 0 -1"/>
-    <limit effort="1000.0" lower="${-pi}" upper="${pi}" velocity="0.5"/>
+    <limit effort="1000.0" lower="${-pi}" upper="${pi}" velocity="10"/>
   </joint>
   <joint name="joint_2" type="revolute">
@@ -124,5 +124,5 @@
     <origin xyz="0 0.0245 0.058952" rpy="${pi/2} ${-pi/2} 0"/>
     <axis xyz="0 0 -1"/>
-    <limit effort="1000.0" lower="${-pi}" upper="${pi}" velocity="0.5"/>
+    <limit effort="1000.0" lower="${-pi}" upper="${pi}" velocity="10"/>
   </joint>
   <joint name="joint_3" type="revolute">
@@ -131,5 +131,5 @@
     <origin xyz="0.409872 0 -0.002" rpy="${pi} 0 ${-pi/2}"/>
     <axis xyz="0 0 -1"/>
-    <limit effort="1000.0" lower="${-3*pi/2}" upper="${pi/2}" velocity="0.5"/>
+    <limit effort="1000.0" lower="${-3*pi/2}" upper="${pi/2}" velocity="10"/>
   </joint>
   <joint name="joint_4" type="revolute">
@@ -138,5 +138,5 @@
     <origin xyz="0.2339 0 -0.014" rpy="0 ${3*pi/2} ${pi}"/>
     <axis xyz="0 0 -1"/>
-    <limit effort="1000.0" lower="${-pi}" upper="${pi}" velocity="0.5"/>
+    <limit effort="1000.0" lower="${-pi}" upper="${pi}" velocity="10"/>
   </joint>
   <joint name="joint_5" type="revolute">
@@ -145,5 +145,5 @@
     <origin xyz="0 0.090 0.083" rpy="${(65*pi)/180} 0 ${pi}"/>
     <axis xyz="0 0 -1"/>
-    <limit effort="1000.0" lower="${-pi}" upper="${pi}" velocity="0.5"/>
+    <limit effort="1000.0" lower="${-pi}" upper="${pi}" velocity="10"/>
   </joint>
 <!--

Commit message: (feat): add POC2 URDF

File: explorer/description/urdf/explorer.urdf.xacro (robot description, xacro)
@@ -3,6 +3,5 @@
   <xacro:arg name="use_ignition" default="false" />
   <xacro:arg name="use_actuator_interface" default="false" />
-  <!-- Import explorer macro -->
-  <xacro:include filename="$(find ros2_control_explorer)/description/urdf/explorer_old_description.urdf.xacro"/>
+  <xacro:arg name="use_POC2" default="false" />
   <xacro:include filename="$(find gripper_pincette)/description/urdf/gripper_pincette_description.urdf.xacro"/>
   <!-- create link fixed to the "world" -->
@@ -16,11 +15,28 @@
     <axis xyz="0 0 1"/>
   </joint>
-  <joint name="joint_6" type="revolute">
-    <parent link="link_5"/>
-    <child link="structure"/>
-    <origin xyz="0 0.090 0.083" rpy="0 ${(65*pi)/180} ${pi/2}"/>
-    <axis xyz="0 0 -1"/>
-    <limit effort="1000.0" lower="${-pi}" upper="${pi}" velocity="10"/>
-  </joint>
+  <xacro:unless value="$(arg use_POC2)">
+    <!-- Import explorer macro -->
+    <xacro:include filename="$(find ros2_control_explorer)/description/urdf/explorer_POC1_description.urdf.xacro"/>
+    <joint name="joint_6" type="revolute">
+      <parent link="link_5"/>
+      <child link="structure"/>
+      <origin xyz="0 0.090 0.083" rpy="0 ${(65*pi)/180} ${pi/2}"/>
+      <axis xyz="0 0 -1"/>
+      <limit effort="1000.0" lower="${-pi}" upper="${pi}" velocity="10"/>
+    </joint>
+    <xacro:explorer_POC1_description/>
+  </xacro:unless>
+  <xacro:if value="$(arg use_POC2)">
+    <!-- Import explorer macro -->
+    <xacro:include filename="$(find ros2_control_explorer)/description/urdf/explorer_POC2_description.urdf.xacro"/>
+    <joint name="joint_6" type="revolute">
+      <parent link="link_5"/>
+      <child link="structure"/>
+      <origin xyz="0 0.1555 -0.027" rpy="${pi/2} 0 ${pi}"/>
+      <axis xyz="0 0 -1"/>
+      <limit effort="1000.0" lower="${-pi}" upper="${pi}" velocity="10"/>
+    </joint>
+    <xacro:explorer_POC2_description/>
+  </xacro:if>
   <joint name="joint-ft_frame" type="fixed">
     <parent link="structure"/>
@@ -38,5 +54,4 @@
     <origin xyz="0 0 0" rpy="0 0 0"/>
   </joint>
-  <xacro:explorer_old_description/>
   <xacro:gripper_pincette/>
   <!-- Import explorer ros2_control description -->

Commit message: (fix): change for POC2 to work properly

File: explorer/description/urdf/explorer.urdf.xacro (robot description, xacro)
@@ -33,7 +33,7 @@
       <parent link="link_5"/>
       <child link="structure"/>
-      <origin xyz="0 0.1555 -0.027" rpy="${pi/2} 0 ${pi}"/>
+      <origin xyz="0 0.1555 -0.027" rpy="${pi/2} ${pi} ${pi}"/>
       <axis xyz="0 0 -1"/>
-      <limit effort="1000.0" lower="${-pi}" upper="${pi}" velocity="10"/>
+      <limit effort="1000.0" lower="-2.97" upper="2.97" velocity="10"/>
     </joint>
     <xacro:explorer_POC2_description/>

File: explorer/description/urdf/explorer_POC2_description.urdf.xacro (robot description, xacro)
@@ -107,5 +107,5 @@
       iyy="1"
       iyz="0"
-      izz="1"
+      izz="1"3 cm de marge hors du PCB et rien dedans pour +-200°
   /> -->
   <link name="ft_frame"/>
@@ -117,5 +117,5 @@
     <origin xyz="0 0 0.0555" rpy="0 0 0"/>
     <axis xyz="0 0 -1"/>
-    <limit effort="1000.0" lower="${-pi}" upper="${pi}" velocity="2.5"/>
+    <limit effort="1000.0" lower="${-pi}" upper="${pi}" velocity="10"/>
   </joint>
   <joint name="joint_2" type="revolute">
@@ -124,5 +124,5 @@
     <origin xyz="0 0.0265 0.058952" rpy="${pi/2} ${-pi/2} 0"/>
     <axis xyz="0 0 -1"/>
-    <limit effort="1000.0" lower="${-pi/2}" upper="${pi/2}" velocity="2.5"/>
+    <limit effort="1000.0" lower="${-pi/2}" upper="${pi/2}" velocity="10"/>
   </joint>
   <joint name="joint_3" type="revolute">
@@ -131,12 +131,12 @@
     <origin xyz="0.413 0 0" rpy="${pi} 0 0"/>
     <axis xyz="0 0 -1"/>
-    <limit effort="1000.0" lower="${-3*pi/2}" upper="${pi/2}" velocity="2.5"/>
+    <limit effort="1000.0" lower="${-3*pi/2}" upper="${pi/2}" velocity="10"/>
   </joint>
   <joint name="joint_4" type="revolute">
     <parent link="link_3"/>
     <child link="link_4"/>
-    <origin xyz="0.1885 0 -0.008" rpy="${pi/2} 0 ${pi/2}"/>
+    <origin xyz="0.1885 0 -0.008" rpy="${pi/2} ${pi} ${pi/2}"/>
     <axis xyz="0 0 -1"/>
-    <limit effort="1000.0" lower="${-pi}" upper="${pi}" velocity="2.5"/>
+    <limit effort="1000.0" lower="${-pi}" upper="${pi}" velocity="10"/>
   </joint>
   <joint name="joint_5" type="revolute">
@@ -145,5 +145,5 @@
     <origin xyz="0 0.0285 0.1" rpy="${pi/2} 0 ${pi}"/>
     <axis xyz="0 0 -1"/>
-    <limit effort="1000.0" lower="${-pi}" upper="${pi}" velocity="2.5"/>
+    <limit effort="1000.0" lower="${-pi}" upper="${pi}" velocity="10"/>
   </joint>
   <!-- <joint name="joint_6" type="revolute">
@@ -152,5 +152,5 @@
     <origin xyz="-0.150049 0 -0.028307" rpy="0 ${-pi/2} 0"/>
     <axis xyz="0 0 1"/>
-    <limit effort="1000.0" lower="${-pi}" upper="${pi}" velocity="2.5"/>
+    <limit effort="1000.0" lower="${-pi}" upper="${pi}" velocity="10"/>
   </joint>
   <joint name="joint-ft_frame" type="fixed">

Commit message: feat: invert actuators directions to match REP103, to macth vesc_firmware after ORTHOPUS-EXPLORER/vesc_firmware@8d13b2e

File: explorer/description/urdf/explorer.urdf.xacro (robot description, xacro)
@@ -26,5 +26,5 @@
       <child link="structure"/>
       <origin xyz="0 0.090 0.083" rpy="0 ${(65*pi)/180} ${pi/2}"/>
-      <axis xyz="0 0 -1"/>
+      <axis xyz="0 0 1"/>
       <limit effort="1000.0" lower="${-pi}" upper="${pi}" velocity="10"/>
     </joint>
@@ -38,5 +38,5 @@
       <child link="structure"/>
       <origin xyz="0 0.1555 -0.027" rpy="${pi/2} ${pi} ${pi}"/>
-      <axis xyz="0 0 -1"/>
+      <axis xyz="0 0 1"/>
       <limit effort="1000.0" lower="-2.97" upper="2.97" velocity="10"/>
     </joint>

File: explorer/description/urdf/explorer_POC2_description.urdf.xacro (robot description, xacro)
@@ -116,5 +116,5 @@
     <child link="link_1"/>
     <origin xyz="0 0 0.0555" rpy="0 0 0"/>
-    <axis xyz="0 0 -1"/>
+    <axis xyz="0 0 1"/>
     <limit effort="1000.0" lower="-2.97" upper="2.97" velocity="10"/>
   </joint>
@@ -123,5 +123,5 @@
     <child link="link_2"/>
     <origin xyz="0 0.0265 0.058952" rpy="${pi/2} ${-pi/2} 0"/>
-    <axis xyz="0 0 -1"/>
+    <axis xyz="0 0 1"/>
     <limit effort="1000.0" lower="-2.14" upper="2.14" velocity="10"/>
   </joint>
@@ -130,5 +130,5 @@
     <child link="link_3"/>
     <origin xyz="0.413 0 0" rpy="${pi} 0 0"/>
-    <axis xyz="0 0 -1"/>
+    <axis xyz="0 0 1"/>
     <limit effort="1000.0" lower="-2.97" upper="2.97" velocity="10"/>
   </joint>
@@ -137,5 +137,5 @@
     <child link="link_4"/>
     <origin xyz="0.1885 0 -0.008" rpy="${pi/2} ${pi} ${pi/2}"/>
-    <axis xyz="0 0 -1"/>
+    <axis xyz="0 0 1"/>
     <limit effort="1000.0" lower="-2.97" upper="2.97" velocity="10"/>
   </joint>
@@ -144,5 +144,5 @@
     <child link="link_5"/>
     <origin xyz="0 0.0285 0.1" rpy="${pi/2} 0 ${pi}"/>
-    <axis xyz="0 0 -1"/>
+    <axis xyz="0 0 1"/>
     <limit effort="1000.0" lower="-1.8" upper="1.8" velocity="10"/>
   </joint>
