Commit message: feat(actuator_standalone): Update to use new vescpp lib

File: actuator_standalone/description/ros2_control/actuator.ros2_control.xacro (robot description, xacro)
@@ -1,5 +1,5 @@
 <?xml version="1.0"?>
 <robot xmlns:xacro="http://www.ros.org/wiki/xacro">
-  <xacro:macro name="actuator_ros2_control" params="name use_ignition:=^|false">
+  <xacro:macro name="actuator_ros2_control" params="name use_ignition:=^|false can_port:=^|vxcan1 can_id:=^|17  host_id:=^|45">
   <ros2_control name="${name}" type="actuator">
     <hardware>
@@ -8,6 +8,9 @@
         </xacro:if>
         <xacro:unless value="${use_ignition}">
-          <plugin>orthopus_ros_interface/HwInterface</plugin>
+          <plugin>orthopus_vesc_interface/VESCInterface</plugin>
         </xacro:unless>
+      <param name="can_port">${can_port}</param>
+      <param name="can_id">${can_id}</param>
+      <param name="host_id">${host_id}</param>
     </hardware>
     <joint name="joint">

File: actuator_standalone/description/urdf/actuator.urdf.xacro (robot description, xacro)
@@ -3,4 +3,7 @@
   <xacro:arg name="use_ignition" default="false" />
   <xacro:arg name="use_actuator_interface" default="false" />
+  <xacro:arg name="can_port" default="vxcan1" />
+  <xacro:arg name="can_id" default="17" />
+  <xacro:arg name="host_id" default="45" />
   <!-- Import actuator macro -->
   <xacro:include filename="$(find ros2_control_actuator)/description/urdf/actuator_description.urdf.xacro"/>
@@ -16,5 +19,5 @@
   <!-- Import actuator ros2_control description -->
  <xacro:include filename="$(find ros2_control_actuator)/description/ros2_control/actuator.ros2_control.xacro" />
-  <xacro:actuator_ros2_control name="actuator" use_ignition="$(arg use_ignition)" />
+  <xacro:actuator_ros2_control name="actuator" use_ignition="$(arg use_ignition)"  can_port="$(arg can_port)" can_id="$(arg can_id)" host_id="$(arg host_id)" />
   <xacro:if value="$(arg use_ignition)">
     <!-- Import Gazebo definitions + plugin -->

Commit message: fix: standalone actuator launch file - support stream rates

File: actuator_standalone/description/ros2_control/actuator.ros2_control.xacro (robot description, xacro)
@@ -1,5 +1,5 @@
 <?xml version="1.0"?>
 <robot xmlns:xacro="http://www.ros.org/wiki/xacro">
-  <xacro:macro name="actuator_ros2_control" params="name use_ignition:=^|false can_port:=^|vxcan1 can_id:=^|17  host_id:=^|45">
+  <xacro:macro name="actuator_ros2_control" params="name use_ignition:=^|false can_port:=^|vxcan1 can_id:=^|17  host_id:=^|45 rt_stream_rate:=^|250 aux_stream_rate:=^|10">
   <ros2_control name="${name}" type="actuator">
     <hardware>
@@ -13,4 +13,6 @@
       <param name="can_id">${can_id}</param>
       <param name="host_id">${host_id}</param>
+      <param name="rt_stream_rate">${rt_stream_rate}</param>
+      <param name="aux_stream_rate">${aux_stream_rate}</param>
     </hardware>
     <joint name="joint">

File: actuator_standalone/description/urdf/actuator.urdf.xacro (robot description, xacro)
@@ -6,4 +6,6 @@
   <xacro:arg name="can_id" default="17" />
   <xacro:arg name="host_id" default="45" />
+  <xacro:arg name="rt_stream_rate" default="250" />
+  <xacro:arg name="aux_stream_rate" default="10" />
   <!-- Import actuator macro -->
   <xacro:include filename="$(find ros2_control_actuator)/description/urdf/actuator_description.urdf.xacro"/>
@@ -19,5 +21,13 @@
   <!-- Import actuator ros2_control description -->
  <xacro:include filename="$(find ros2_control_actuator)/description/ros2_control/actuator.ros2_control.xacro" />
-  <xacro:actuator_ros2_control name="actuator" use_ignition="$(arg use_ignition)"  can_port="$(arg can_port)" can_id="$(arg can_id)" host_id="$(arg host_id)" />
+  <xacro:actuator_ros2_control
+    name="actuator"
+    use_ignition="$(arg use_ignition)"
+    can_port="$(arg can_port)"
+    can_id="$(arg can_id)"
+    host_id="$(arg host_id)"
+    rt_stream_rate="$(arg rt_stream_rate)"
+    aux_stream_rate="$(arg aux_stream_rate)"
+  />
   <xacro:if value="$(arg use_ignition)">
     <!-- Import Gazebo definitions + plugin -->
