Commit message: fix: gripper command stream rate was changed from 50 to 10, restoring previous value

File: actuator_standalone/description/ros2_control/actuator.ros2_control.xacro (robot description, xacro)
@@ -1,5 +1,5 @@
 <?xml version="1.0"?>
 <robot xmlns:xacro="http://www.ros.org/wiki/xacro">
-  <xacro:macro name="actuator_ros2_control" params="name use_ignition:=^|false can_port:=^|vxcan1 can_id:=^|17  host_id:=^|45 rt_stream_rate:=^|250 aux_stream_rate:=^|10">
+  <xacro:macro name="actuator_ros2_control" params="name use_ignition:=^|false can_port:=^|vxcan1 can_id:=^|17  host_id:=^|45 rt_stream_rate aux_config_stream_rate aux_servo_stream_rate">
   <ros2_control name="${name}" type="actuator">
     <hardware>
@@ -14,5 +14,6 @@
       <param name="host_id">${host_id}</param>
       <param name="rt_stream_rate">${rt_stream_rate}</param>
-      <param name="aux_stream_rate">${aux_stream_rate}</param>
+      <param name="aux_config_stream_rate">${aux_config_stream_rate}</param>
+      <param name="aux_servo_stream_rate">${aux_servo_stream_rate}</param>
     </hardware>
     <joint name="joint">

File: actuator_standalone/description/urdf/actuator.urdf.xacro (robot description, xacro)
@@ -7,5 +7,6 @@
   <xacro:arg name="host_id" default="45" />
   <xacro:arg name="rt_stream_rate" default="250" />
-  <xacro:arg name="aux_stream_rate" default="10" />
+  <xacro:arg name="aux_config_stream_rate" default="10" />
+  <xacro:arg name="aux_servo_stream_rate" default="50" />
   <!-- Import actuator macro -->
   <xacro:include filename="$(find ros2_control_actuator)/description/urdf/actuator_description.urdf.xacro"/>
@@ -28,5 +29,6 @@
     host_id="$(arg host_id)"
     rt_stream_rate="$(arg rt_stream_rate)"
-    aux_stream_rate="$(arg aux_stream_rate)"
+    aux_config_stream_rate="$(arg aux_config_stream_rate)"
+    aux_servo_stream_rate="$(arg aux_servo_stream_rate)"
   />
   <xacro:if value="$(arg use_ignition)">

File: explorer_description/ros2_control/explorer_actuators.ros2_control.xacro (robot description, xacro)
@@ -2,5 +2,5 @@
 <robot xmlns:xacro="http://www.ros.org/wiki/xacro">
   <xacro:include filename="$(find explorer_description)/urdf/explorer_joints.xacro" />
-  <xacro:macro name="explorer_ros2_control" params="name can_port:=^|can0  host_id:=^|45 rt_stream_rate:=^|250 aux_servo_stream_rate:=^|10 aux_config_stream_rate:=^|10">
+  <xacro:macro name="explorer_ros2_control" params="name can_port:=^|can0  host_id:=^|45 rt_stream_rate aux_servo_stream_rate aux_config_stream_rate">
     <xacro:macro name="hw_intf_params">
       <plugin>orthopus_vesc_interface/VESCInterface</plugin>

File: explorer_description/urdf/explorer.urdf.xacro (robot description, xacro)
@@ -10,5 +10,5 @@
     <xacro:arg name="host_id" default="45" />
     <xacro:arg name="rt_stream_rate" default="250" />
-    <xacro:arg name="aux_servo_stream_rate" default="20" />
+    <xacro:arg name="aux_servo_stream_rate" default="50" />
     <xacro:arg name="aux_config_stream_rate" default="10" />
     <!-- endif -->
