Commit message: refactor: move explorer_description

File: explorer_description/ros2_control/explorer.ros2_control.xacro (robot description, xacro)
@@ -2,5 +2,5 @@
 <robot xmlns:xacro="http://www.ros.org/wiki/xacro">
   <xacro:macro name="explorer_ros2_control" params="name use_ignition:=^|false can_port:=^|vxcan1 host_id:=^|45">
-    <xacro:include filename="$(find ros2_control_explorer)/explorer_description/urdf/explorer_joints.xacro" />
+    <xacro:include filename="$(find explorer_description)/urdf/explorer_joints.xacro" />
     <ros2_control name="${name}" type="system">
       <hardware>

File: explorer_description/ros2_control/explorer_actuators.ros2_control.xacro (robot description, xacro)
@@ -1,5 +1,5 @@
 <?xml version="1.0"?>
 <robot xmlns:xacro="http://www.ros.org/wiki/xacro">
-  <xacro:include filename="$(find ros2_control_explorer)/explorer_description/urdf/explorer_joints.xacro" />
+  <xacro:include filename="$(find explorer_description)/urdf/explorer_joints.xacro" />
   <xacro:macro name="explorer_ros2_control" params="name use_ignition:=^|false can_port:=^|vxcan1  host_id:=^|45 rt_stream_rate:=^|250 aux_stream_rate:=^|10">
     <xacro:macro name="hw_intf_params">

File: explorer_description/urdf/explorer.urdf.xacro (robot description, xacro)
@@ -21,5 +21,5 @@
   <xacro:unless value="$(arg use_POC2)">
     <!-- Import explorer macro -->
-    <xacro:include filename="$(find ros2_control_explorer)/explorer_description/urdf/explorer_POC1_description.urdf.xacro"/>
+    <xacro:include filename="$(find explorer_description)/urdf/explorer_POC1_description.urdf.xacro"/>
     <joint name="joint_6" type="revolute">
       <parent link="link_5"/>
@@ -33,5 +33,5 @@
   <xacro:if value="$(arg use_POC2)">
     <!-- Import explorer macro -->
-    <xacro:include filename="$(find ros2_control_explorer)/explorer_description/urdf/explorer_POC2_description.urdf.xacro"/>
+    <xacro:include filename="$(find explorer_description)/urdf/explorer_POC2_description.urdf.xacro"/>
     <joint name="joint_6" type="revolute">
       <parent link="link_5"/>
@@ -61,9 +61,9 @@
   <!-- Import explorer ros2_control description -->
   <xacro:unless value="$(arg use_actuator_interface)">
-    <xacro:include filename="$(find ros2_control_explorer)/explorer_description/ros2_control/explorer.ros2_control.xacro" />
+    <xacro:include filename="$(find explorer_description)/ros2_control/explorer.ros2_control.xacro" />
     <xacro:explorer_ros2_control name="explorer" use_ignition="$(arg use_ignition)" />
   </xacro:unless>
   <xacro:if value="$(arg use_actuator_interface)">
-    <xacro:include filename="$(find ros2_control_explorer)/explorer_description/ros2_control/explorer_actuators.ros2_control.xacro" />
+    <xacro:include filename="$(find explorer_description)/ros2_control/explorer_actuators.ros2_control.xacro" />
     <xacro:explorer_ros2_control
       name="explorer"
@@ -77,5 +77,5 @@
   <xacro:if value="$(arg use_ignition)">
     <!-- Import Gazebo definitions + plugin -->
-    <xacro:include filename="$(find ros2_control_explorer)/explorer_description/gazebo/explorer.gazebo.xacro" />
+    <xacro:include filename="$(find explorer_description)/gazebo/explorer.gazebo.xacro" />
     <xacro:explorer_gazebo/>
   </xacro:if>

File: explorer_description/urdf/explorer_POC1_description.urdf.xacro (robot description, xacro)
@@ -3,10 +3,10 @@
   <xacro:macro name="explorer_POC1_description">
   <!-- helper macro -->
-  <xacro:include filename="$(find ros2_control_explorer)/explorer_description/urdf/inc/create_link.xacro"/>
+  <xacro:include filename="$(find explorer_description)/urdf/inc/create_link.xacro"/>
   <xacro:create_link
       link_name="base_link"
       xyz_offset="0 0 0"
       rpy_offset="0 0 0"
-      mesh_package="ros2_control_explorer"
+      mesh_package="explorer_description"
       mesh_name="base_link_POC1"
       xyz_mass="0.000045 0.000001 0.026873"
@@ -23,5 +23,5 @@
       xyz_offset="0 0 0"
       rpy_offset="0 0 0"
-      mesh_package="ros2_control_explorer"
+      mesh_package="explorer_description"
       mesh_name="link1_POC1"
       xyz_mass="-0.000001 0.02935 0.029854"
@@ -38,5 +38,5 @@
       xyz_offset="0 0 0"
       rpy_offset="0 0 0"
-      mesh_package="ros2_control_explorer"
+      mesh_package="explorer_description"
       mesh_name="link2_POC1"
       xyz_mass="0.204774 0.000012 0.057505"
@@ -53,5 +53,5 @@
       xyz_offset="0 0 0"
       rpy_offset="0 0 0"
-      mesh_package="ros2_control_explorer"
+      mesh_package="explorer_description"
       mesh_name="link3_POC1"
       xyz_mass="0.138064 -0.000019  -0.007584"
@@ -68,5 +68,5 @@
       xyz_offset="0 0 0"
       rpy_offset="0 0 0"
-      mesh_package="ros2_control_explorer"
+      mesh_package="explorer_description"
       mesh_name="link4_POC1"
       xyz_mass="0.000006 0.044695  0.057883"
@@ -83,5 +83,5 @@
       xyz_offset="0 0 0"
       rpy_offset="0 0 0"
-      mesh_package="ros2_control_explorer"
+      mesh_package="explorer_description"
       mesh_name="link5_POC1"
       xyz_mass="0.000006 0.044695  0.057883"
@@ -98,5 +98,5 @@
       xyz_offset="0 0 0"
       rpy_offset="0 0 0"
-      mesh_package="ros2_control_explorer"
+      mesh_package="explorer_description"
       mesh_name="gripper"
       xyz_mass="0.00224 -0.000032 0.077277"

File: explorer_description/urdf/explorer_POC2_description.urdf.xacro (robot description, xacro)
@@ -3,10 +3,10 @@
   <xacro:macro name="explorer_POC2_description">
   <!-- helper macro -->
-  <xacro:include filename="$(find ros2_control_explorer)/explorer_description/urdf/inc/create_link.xacro"/>
+  <xacro:include filename="$(find explorer_description)/urdf/inc/create_link.xacro"/>
   <xacro:create_link
       link_name="base_link"
       xyz_offset="0 0 0"
       rpy_offset="0 0 0"
-      mesh_package="ros2_control_explorer"
+      mesh_package="explorer_description"
       mesh_name="base_link_POC2"
       xyz_mass="0 0 0"
@@ -23,5 +23,5 @@
       xyz_offset="0 0 0"
       rpy_offset="0 0 0"
-      mesh_package="ros2_control_explorer"
+      mesh_package="explorer_description"
       mesh_name="link0_POC2"
       xyz_mass="0 0 0"
@@ -38,5 +38,5 @@
       xyz_offset="0 0 0"
       rpy_offset="0 0 0"
-      mesh_package="ros2_control_explorer"
+      mesh_package="explorer_description"
       mesh_name="link1_POC2"
       xyz_mass="0 0 0"
@@ -53,5 +53,5 @@
       xyz_offset="0 0 0"
       rpy_offset="0 0 0"
-      mesh_package="ros2_control_explorer"
+      mesh_package="explorer_description"
       mesh_name="link2_POC2"
       xyz_mass="0 0 0"
@@ -68,5 +68,5 @@
       xyz_offset="0 0 0"
       rpy_offset="0 0 0"
-      mesh_package="ros2_control_explorer"
+      mesh_package="explorer_description"
       mesh_name="link3_POC2"
       xyz_mass="0 0 0"
@@ -83,5 +83,5 @@
       xyz_offset="0 0 0"
       rpy_offset="0 0 0"
-      mesh_package="ros2_control_explorer"
+      mesh_package="explorer_description"
       mesh_name="link4_POC2"
       xyz_mass="0 0 0"
@@ -98,5 +98,5 @@
       xyz_offset="0 0 0"
       rpy_offset="0 0 0"
-      mesh_package="ros2_control_explorer"
+      mesh_package="explorer_description"
       mesh_name="gripper"
       xyz_mass="0 0 0"

File: explorer_description/urdf/inc/create_link.xacro (robot description, xacro)
@@ -19,5 +19,5 @@
         <origin xyz="${xyz_offset}" rpy="${rpy_offset}"/>
         <geometry>
-          <mesh filename="file://$(find ${mesh_package})/explorer_description/meshes/visual/${mesh_name}.dae" scale="0.001 0.001 0.001"/>
+          <mesh filename="file://$(find ${mesh_package})/meshes/visual/${mesh_name}.dae" scale="0.001 0.001 0.001"/>
         </geometry>
       </visual>
@@ -25,5 +25,5 @@
         <origin xyz="${xyz_offset}" rpy="${rpy_offset}"/>
         <geometry>
-          <mesh filename="file://$(find ${mesh_package})/explorer_description/meshes/collision/${mesh_name}.stl" scale="0.001 0.001 0.001"/>
+          <mesh filename="file://$(find ${mesh_package})/meshes/collision/${mesh_name}.stl" scale="0.001 0.001 0.001"/>
         </geometry>
       </collision>
