Commit message: feat: Add impedance_control_[damping|stiffness] setup in orthopus_vesc_interface from topic input

File: explorer_description/ros2_control/explorer_actuators.ros2_control.xacro (robot description, xacro)
@@ -2,5 +2,5 @@
 <robot xmlns:xacro="http://www.ros.org/wiki/xacro">
   <xacro:include filename="$(find explorer_description)/urdf/explorer_joints.xacro" />
-  <xacro:macro name="explorer_ros2_control" params="name can_port:=^|vxcan1  host_id:=^|45 rt_stream_rate:=^|250 aux_stream_rate:=^|10">
+  <xacro:macro name="explorer_ros2_control" params="name can_port:=^|vxcan1  host_id:=^|45 rt_stream_rate:=^|250 aux_servo_stream_rate:=^|10 aux_config_stream_rate:=^|10">
     <xacro:macro name="hw_intf_params">
       <plugin>orthopus_vesc_interface/VESCInterface</plugin>
@@ -8,5 +8,6 @@
       <param name="can_port">${can_port}</param>
       <param name="rt_stream_rate">${rt_stream_rate}</param>
-      <param name="aux_stream_rate">${aux_stream_rate}</param>
+      <param name="aux_servo_stream_rate">${aux_servo_stream_rate}</param>
+      <param name="aux_config_stream_rate">${aux_config_stream_rate}</param>
       <param name="default_mode">position</param>
     </xacro:macro>

File: explorer_description/urdf/explorer.urdf.xacro (robot description, xacro)
@@ -10,5 +10,6 @@
     <xacro:arg name="host_id" default="45" />
     <xacro:arg name="rt_stream_rate" default="250" />
-    <xacro:arg name="aux_stream_rate" default="50" />
+    <xacro:arg name="aux_servo_stream_rate" default="10" />
+    <xacro:arg name="aux_config_stream_rate" default="10" />
     <!-- endif -->
   <xacro:include filename="$(find gripper_pincette)/description/urdf/gripper_pincette_description.urdf.xacro"/>
@@ -90,5 +91,6 @@
       host_id="$(arg host_id)"
       rt_stream_rate="$(arg rt_stream_rate)"
-      aux_stream_rate="$(arg aux_stream_rate)"
+      aux_servo_stream_rate="$(arg aux_servo_stream_rate)"
+      aux_config_stream_rate="$(arg aux_config_stream_rate)"
     />
   </xacro:unless>

Commit message: dev: allow virtual can interface to be used for simulation

File: explorer_description/ros2_control/explorer_actuators.ros2_control.xacro (robot description, xacro)
@@ -2,5 +2,5 @@
 <robot xmlns:xacro="http://www.ros.org/wiki/xacro">
   <xacro:include filename="$(find explorer_description)/urdf/explorer_joints.xacro" />
-  <xacro:macro name="explorer_ros2_control" params="name can_port:=^|vxcan1  host_id:=^|45 rt_stream_rate:=^|250 aux_servo_stream_rate:=^|10 aux_config_stream_rate:=^|10">
+  <xacro:macro name="explorer_ros2_control" params="name can_port:=^|can0  host_id:=^|45 rt_stream_rate:=^|250 aux_servo_stream_rate:=^|10 aux_config_stream_rate:=^|10">
     <xacro:macro name="hw_intf_params">
       <plugin>orthopus_vesc_interface/VESCInterface</plugin>

File: explorer_description/urdf/explorer.urdf.xacro (robot description, xacro)
@@ -7,5 +7,5 @@
     <xacro:arg name="use_ignition" default="true" />
     <!-- else -->
-    <xacro:arg name="can_port" default="vxcan1" />
+    <xacro:arg name="can_port" default="can0" />
     <xacro:arg name="host_id" default="45" />
     <xacro:arg name="rt_stream_rate" default="250" />

Commit message: dev: add support for new ros param "debug" (set debug logger level)

File: explorer_description/ros2_control/explorer_actuators.ros2_control.xacro (robot description, xacro)
@@ -2,5 +2,5 @@
 <robot xmlns:xacro="http://www.ros.org/wiki/xacro">
   <xacro:include filename="$(find explorer_description)/urdf/explorer_joints.xacro" />
-  <xacro:macro name="explorer_ros2_control" params="name can_port:=^|can0  host_id:=^|45 rt_stream_rate aux_servo_stream_rate aux_config_stream_rate">
+  <xacro:macro name="explorer_ros2_control" params="name can_port:=^|can0  host_id:=^|45 rt_stream_rate aux_servo_stream_rate aux_config_stream_rate debug:=^|false">
     <xacro:macro name="hw_intf_params">
       <plugin>orthopus_vesc_interface/VESCInterface</plugin>
@@ -11,4 +11,5 @@
       <param name="aux_config_stream_rate">${aux_config_stream_rate}</param>
       <param name="default_mode">position</param>
+      <param name="debug">${debug}</param>
     </xacro:macro>
   <!-- ROS2 Control -->

Commit message: dev: add support for new ros param "debug" (set debug logger level)

File: explorer_description/ros2_control/explorer_actuators.ros2_control.xacro (robot description, xacro)
@@ -2,5 +2,5 @@
 <robot xmlns:xacro="http://www.ros.org/wiki/xacro">
   <xacro:include filename="$(find explorer_description)/urdf/explorer_joints.xacro" />
-  <xacro:macro name="explorer_ros2_control" params="name can_port:=^|can0  host_id:=^|45 rt_stream_rate:=^|250 aux_servo_stream_rate:=^|10 aux_config_stream_rate:=^|10">
+  <xacro:macro name="explorer_ros2_control" params="name can_port:=^|can0  host_id:=^|45 rt_stream_rate:=^|250 aux_servo_stream_rate:=^|10 aux_config_stream_rate:=^|10 debug:=^|false">
     <xacro:macro name="hw_intf_params">
       <plugin>orthopus_vesc_interface/VESCInterface</plugin>
@@ -11,4 +11,5 @@
       <param name="aux_config_stream_rate">${aux_config_stream_rate}</param>
       <param name="default_mode">position</param>
+      <param name="debug">${debug}</param>
     </xacro:macro>
   <!-- ROS2 Control -->

File: explorer_description/urdf/explorer.urdf.xacro (robot description, xacro)
@@ -4,4 +4,5 @@
   <xacro:arg name="simulation" default="false" />
   <xacro:arg name="robot_controller_config" default="controller" />
+  <xacro:arg name="debug" default="false" />
     <!-- if Simulation-->
     <xacro:arg name="use_ignition" default="true" />
@@ -93,4 +94,5 @@
       aux_servo_stream_rate="$(arg aux_servo_stream_rate)"
       aux_config_stream_rate="$(arg aux_config_stream_rate)"
+      debug="$(arg debug)"
     />
   </xacro:unless>

Commit message: Dev/impedance control (#34)
* refactor: delete unused 'controller' modes from  explorer_multi_intf_controller

* refactor: delete unused QoS settings (and set by default)

* refactor: format + fix linter issues in explorer_command_controllers

* refactor: add share/simulation/hardware reusable methods to reduce launch code duplication

* refactor: add new launch files to explorer_bringup for custom_controller + remove old multi_intf* launch files

* dev: First base of custom controller added for impedance control

* dev: Add effort interface to urdf files + add controller type (custom / controller)

* dev: Add simulation support for explorer_command_controllers->custom_controller

* dev: set actuator mode on explorer_command_controllers->custom_controller startup

* dev: add impedance damping / stiffness setup on custom_controller startup

* dev: Fix several issues related to mode0 + impedance

* dev: Fix device issue related to Docker / permissions

* dev: allow parametrable controller switch in command_node

* dev: custom_controller deal properlly with ros2 control switch

* dev: remove unused launch file

* dev: Fix issue in explorer_custom_controller regarding topic input size check

* feat: Add impedance_control_[damping|stiffness] setup in orthopus_vesc_interface from topic input + no longer start thread streaming manually

* dev: allow virtual can interface to be used for simulation

* fix: prevent crash from web_gui_node on CTRL+C + adapt to refactor

* dev: Add base dependencies to Docker for using gdb

* feat: base impedance config

* dev: changes Docker user to root for dev (easier management / will allow gdb debugging)

* fix: setMode / cmd wasn't working properly inside custom controller, switched from cmd to config topic and stores setMode clients to prevents ROS warning for sender

* fix: issue when custom_controller gets activated more than once (joints gets added continuously)

* dev: try to fix gripper issue by increasing servo stream rate

* dev: fix devcontainer git dubious ownership issue

* fix: gripper command stream rate was changed from 50 to 10, restoring previous value

* feat: impedance control scripts and doc

* dev: update submodule libs/orthopus_vesc to main

---------

Co-authored-by: Thomas Solatges <thomas.solatges@orthopus.com>
Co-authored-by: Thomas Solatges <thomas@solatges.fr>

File: explorer_description/ros2_control/explorer_actuators.ros2_control.xacro (robot description, xacro)
@@ -2,5 +2,5 @@
 <robot xmlns:xacro="http://www.ros.org/wiki/xacro">
   <xacro:include filename="$(find explorer_description)/urdf/explorer_joints.xacro" />
-  <xacro:macro name="explorer_ros2_control" params="name can_port:=^|vxcan1  host_id:=^|45 rt_stream_rate:=^|250 aux_stream_rate:=^|10">
+  <xacro:macro name="explorer_ros2_control" params="name can_port:=^|can0  host_id:=^|45 rt_stream_rate aux_servo_stream_rate aux_config_stream_rate">
     <xacro:macro name="hw_intf_params">
       <plugin>orthopus_vesc_interface/VESCInterface</plugin>
@@ -8,5 +8,6 @@
       <param name="can_port">${can_port}</param>
       <param name="rt_stream_rate">${rt_stream_rate}</param>
-      <param name="aux_stream_rate">${aux_stream_rate}</param>
+      <param name="aux_servo_stream_rate">${aux_servo_stream_rate}</param>
+      <param name="aux_config_stream_rate">${aux_config_stream_rate}</param>
       <param name="default_mode">position</param>
     </xacro:macro>

File: explorer_description/urdf/explorer.urdf.xacro (robot description, xacro)
@@ -3,11 +3,13 @@
   <xacro:arg name="use_POC2" default="false" />
   <xacro:arg name="simulation" default="false" />
+  <xacro:arg name="robot_controller_config" default="controller" />
     <!-- if Simulation-->
     <xacro:arg name="use_ignition" default="true" />
     <!-- else -->
-    <xacro:arg name="can_port" default="vxcan1" />
+    <xacro:arg name="can_port" default="can0" />
     <xacro:arg name="host_id" default="45" />
     <xacro:arg name="rt_stream_rate" default="250" />
-    <xacro:arg name="aux_stream_rate" default="50" />
+    <xacro:arg name="aux_servo_stream_rate" default="50" />
+    <xacro:arg name="aux_config_stream_rate" default="10" />
     <!-- endif -->
   <xacro:include filename="$(find gripper_pincette)/description/urdf/gripper_pincette_description.urdf.xacro"/>
@@ -80,5 +82,5 @@
   <xacro:if value="$(arg simulation)">
     <xacro:include filename="$(find explorer_description)/ros2_control/explorer_simulation.ros2_control.xacro" />
-    <xacro:explorer_ros2_control name="explorer" use_ignition="$(arg use_ignition)" />
+    <xacro:explorer_ros2_control name="explorer" use_ignition="$(arg use_ignition)" robot_controller_config="$(arg robot_controller_config)"/>
   </xacro:if>
   <xacro:unless value="$(arg simulation)">
@@ -89,5 +91,6 @@
       host_id="$(arg host_id)"
       rt_stream_rate="$(arg rt_stream_rate)"
-      aux_stream_rate="$(arg aux_stream_rate)"
+      aux_servo_stream_rate="$(arg aux_servo_stream_rate)"
+      aux_config_stream_rate="$(arg aux_config_stream_rate)"
     />
   </xacro:unless>

Commit message: fix: update last command updated time in write method in orthopus_vesc_interface

File: explorer_description/ros2_control/explorer_actuators.ros2_control.xacro (robot description, xacro)
@@ -2,5 +2,5 @@
 <robot xmlns:xacro="http://www.ros.org/wiki/xacro">
   <xacro:include filename="$(find explorer_description)/urdf/explorer_joints.xacro" />
-  <xacro:macro name="explorer_ros2_control" params="name can_port:=^|can0  host_id:=^|45 rt_stream_rate aux_servo_stream_rate aux_config_stream_rate debug:=^|false">
+  <xacro:macro name="explorer_ros2_control" params="name can_port:=^|can0  host_id:=^|45 rt_stream_rate aux_servo_stream_rate aux_config_stream_rate debug:=^|false can_write_failures_threshold:=^|5">
     <xacro:macro name="hw_intf_params">
       <plugin>orthopus_vesc_interface/VESCInterface</plugin>
@@ -12,4 +12,5 @@
       <param name="default_mode">position</param>
       <param name="debug">${debug}</param>
+      <param name="can_write_failures_threshold">${can_write_failures_threshold}</param>
     </xacro:macro>
   <!-- ROS2 Control -->
