Commit message: feat: allow proper control in frame world or tool, selectable with parameter

File: explorer_description/urdf/explorer.urdf.xacro (robot description, xacro)
@@ -59,5 +59,5 @@
     <parent link="ft_frame"/>
     <child link="tool0"/>
-    <origin xyz="0 0 0" rpy="0 0 0"/>
+    <origin xyz="0 0 0" rpy="0 ${-pi/2} 0"/>
   </joint>
   <xacro:gripper_pincette/>

Commit message: fix: place tool frame alligned with last actuator - simplifies control in tool frame (roll = J6)

File: explorer_description/urdf/explorer.urdf.xacro (robot description, xacro)
@@ -59,5 +59,5 @@
     <parent link="ft_frame"/>
     <child link="tool0"/>
-    <origin xyz="0 0 0" rpy="0 ${-pi/2} 0"/>
+    <origin xyz="-0.011 0 0" rpy="0 ${-pi/2} 0"/>
   </joint>
   <xacro:gripper_pincette/>

Commit message: feat: add drink frames and proper control to control new tools

File: explorer_description/urdf/explorer.urdf.xacro (robot description, xacro)
@@ -61,4 +61,19 @@
     <origin xyz="-0.011 0 0" rpy="0 ${-pi/2} 0"/>
   </joint>
+  <!-- Additional tool frames with lateral offsets for different drink sizes -->
+  <link name="drink_small"/>
+  <link name="drink_big"/>
+  <joint name="joint-drink-small" type="fixed">
+    <parent link="tool0"/>
+    <child link="drink_small"/>
+    <!-- Lateral shift: 30mm in Y direction for small drinks -->
+    <origin xyz="0 -0.035 0.035" rpy="0 0 0"/>
+  </joint>
+  <joint name="joint-drink-big" type="fixed">
+    <parent link="tool0"/>
+    <child link="drink_big"/>
+    <!-- Lateral shift: 60mm in Y direction for big drinks -->
+    <origin xyz="0 -0.045 0.045" rpy="0 0 0"/>
+  </joint>
   <xacro:gripper_pincette/>
   <!-- Import explorer ros2_control description -->

Commit message: feat - update xacro with real velocity limits values

File: explorer_description/urdf/explorer.urdf.xacro (robot description, xacro)
@@ -43,5 +43,5 @@
       <origin xyz="0 0.1555 -0.027" rpy="${pi/2} ${pi} ${pi}"/>
       <axis xyz="0 0 1"/>
-      <limit effort="1000.0" lower="-2.97" upper="2.97" velocity="10"/>
+      <limit effort="1000.0" lower="-2.97" upper="2.97" velocity="25"/>
     </joint>
     <xacro:explorer_POC2_description/>

File: explorer_description/urdf/explorer_POC2_description.urdf.xacro (robot description, xacro)
@@ -117,5 +117,5 @@
     <origin xyz="0 0 0.0555" rpy="0 0 0"/>
     <axis xyz="0 0 1"/>
-    <limit effort="1000.0" lower="-2.97" upper="2.97" velocity="10"/>
+    <limit effort="1000.0" lower="-2.97" upper="2.97" velocity="25"/>
   </joint>
   <joint name="joint_2" type="revolute">
@@ -124,5 +124,5 @@
     <origin xyz="0 0.0265 0.058952" rpy="${pi/2} ${-pi/2} 0"/>
     <axis xyz="0 0 1"/>
-    <limit effort="1000.0" lower="-2.14" upper="2.14" velocity="10"/>
+    <limit effort="1000.0" lower="-2.14" upper="2.14" velocity="25"/>
   </joint>
   <joint name="joint_3" type="revolute">
@@ -131,5 +131,5 @@
     <origin xyz="0.413 0 0" rpy="${pi} 0 0"/>
     <axis xyz="0 0 1"/>
-    <limit effort="1000.0" lower="-2.97" upper="2.97" velocity="10"/>
+    <limit effort="1000.0" lower="-2.97" upper="2.97" velocity="25"/>
   </joint>
   <joint name="joint_4" type="revolute">
@@ -138,5 +138,5 @@
     <origin xyz="0.1885 0 -0.008" rpy="${pi/2} ${pi} ${pi/2}"/>
     <axis xyz="0 0 1"/>
-    <limit effort="1000.0" lower="-2.97" upper="2.97" velocity="10"/>
+    <limit effort="1000.0" lower="-2.97" upper="2.97" velocity="25"/>
   </joint>
   <joint name="joint_5" type="revolute">
@@ -145,5 +145,5 @@
     <origin xyz="0 0.0285 0.1" rpy="${pi/2} 0 ${pi}"/>
     <axis xyz="0 0 1"/>
-    <limit effort="1000.0" lower="-1.8" upper="1.8" velocity="10"/>
+    <limit effort="1000.0" lower="-1.8" upper="1.8" velocity="25"/>
   </joint>
   <!-- <joint name="joint_6" type="revolute">

File: explorer_description/urdf/explorer_joints.xacro (robot description, xacro)
@@ -46,5 +46,5 @@
         </command_interface>
         <state_interface name="position">
-          <param name="initial_value">2.91</param>
+          <param name="initial_value">2.5</param>
         </state_interface>
         <state_interface name="velocity"/>
