Commit message: fix: gripper command sign was inverted in constrast of real servo gripper so URDF was adapted

File: explorer_description/urdf/explorer_joints.xacro (robot description, xacro)
@@ -145,5 +145,6 @@
         </command_interface-->
         <state_interface name="position">
-          <param name="initial_value">0.0</param>
+          <!-- Start open: 0 = closed, 1 = open -->
+          <param name="initial_value">1.0</param>
         </state_interface>
         <!--state_interface name="velocity"/-->
@@ -153,5 +154,6 @@
       <joint name="right_external_rod_joint">
         <param name="mimic">right_finger_joint</param>
-        <param name="multiplier">-1</param>
+        <param name="multiplier">1</param>
+        <param name="offset">-1.05</param>
         <state_interface name="position"/>
         <!--state_interface name="velocity"/-->
@@ -159,5 +161,6 @@
       <joint name="right_fingertip_joint">
         <param name="mimic">right_finger_joint</param>
-        <param name="multiplier">-1</param>
+        <param name="multiplier">1</param>
+        <param name="offset">-1.05</param>
         <state_interface name="position"/>
         <!--state_interface name="velocity"/-->
@@ -165,5 +168,6 @@
       <joint name="left_finger_joint">
         <param name="mimic">right_finger_joint</param>
-        <param name="multiplier">-1</param>
+        <param name="multiplier">1</param>
+        <param name="offset">-1.05</param>
         <state_interface name="position"/>
         <!--state_interface name="velocity"/-->
@@ -171,5 +175,6 @@
       <joint name="left_external_rod_joint">
         <param name="mimic">right_finger_joint</param>
-        <param name="multiplier">-1</param>
+        <param name="multiplier">1</param>
+        <param name="offset">-1.05</param>
         <state_interface name="position"/>
         <!--state_interface name="velocity"/-->
@@ -177,5 +182,6 @@
       <joint name="left_fingertip_joint">
         <param name="mimic">right_finger_joint</param>
-        <param name="multiplier">-1</param>
+        <param name="multiplier">1</param>
+        <param name="offset">-1.05</param>
         <state_interface name="position"/>
         <!--state_interface name="velocity"/-->

File: gripper_pincette/description/ros2_control/gripper_pincette.ros2_control.xacro (robot description, xacro)
@@ -8,5 +8,8 @@
       <joint name="right_finger_joint">
         <command_interface name="position"/>
-        <state_interface name="position"/>
+        <state_interface name="position">
+          <!-- Start open: 0 = closed, 1 = open -->
+          <param name="initial_value">1.0</param>
+        </state_interface>
         <state_interface name="velocity"/>
         <state_interface name="effort"/>
@@ -14,5 +17,6 @@
       <joint name="right_external_rod_joint">
         <param name="mimic">right_finger_joint</param>
-        <param name="multiplier">-1</param>
+        <param name="multiplier">1</param>
+        <param name="offset">-1.05</param>
         <command_interface name="position"/>
         <state_interface name="position"/>
@@ -22,5 +26,6 @@
       <joint name="right_fingertip_joint">
         <param name="mimic">right_finger_joint</param>
-        <param name="multiplier">-1</param>
+        <param name="multiplier">1</param>
+        <param name="offset">-1.05</param>
         <command_interface name="position"/>
         <state_interface name="position"/>
@@ -30,5 +35,6 @@
       <joint name="left_finger_joint">
         <param name="mimic">right_finger_joint</param>
-        <param name="multiplier">-1</param>
+        <param name="multiplier">1</param>
+        <param name="offset">-1.05</param>
         <command_interface name="position"/>
         <state_interface name="position"/>
@@ -38,5 +44,6 @@
       <joint name="left_external_rod_joint">
         <param name="mimic">right_finger_joint</param>
-        <param name="multiplier">-1</param>
+        <param name="multiplier">1</param>
+        <param name="offset">-1.05</param>
         <command_interface name="position"/>
         <state_interface name="position"/>
@@ -46,5 +53,6 @@
       <joint name="left_fingertip_joint">
         <param name="mimic">right_finger_joint</param>
-        <param name="multiplier">-1</param>
+        <param name="multiplier">1</param>
+        <param name="offset">-1.05</param>
         <command_interface name="position"/>
         <state_interface name="position"/>

File: gripper_pincette/description/urdf/gripper_pincette_description.urdf.xacro (robot description, xacro)
@@ -225,13 +225,23 @@
     <origin xyz="-0.002 0 0.101" rpy="0 -1.57 0"/>
   </joint>
+  <!-- right_finger_joint follows the real servo convention:
+         value 0 = gripper closed, value increases = gripper opens (positive velocity opens).
+       Prior: The original model used the opposite convention:
+         rpy="0 -1.57 0", axis="0 0 1", angle 0 = open, angle 1.05 = closed.
+       To reverse the direction while keeping the same physical range [0, 1.05],
+       the joint maps its value q to the original angle with: original_angle = 1.05 - q
+         - axis flipped to "0 0 -1"           -> gives the "-q" part
+         - origin rotated by 1.05 rad about z -> gives the "+1.05" part
+       New rpy = rpy(0, -1.57, 0) followed by a 1.05 rad rotation about the joint z axis.
+  -->
   <joint name="right_finger_joint" type="revolute">
     <parent link="structure"/>
     <child link="right_finger_first_phalanx"/>
-    <origin xyz="0.015 -0.038 0.1015" rpy="0 -1.57 0"/>
-    <axis xyz="0 0 1"/>
+    <origin xyz="0.015 -0.038 0.1015" rpy="-1.569878 -0.520796 1.570340"/>
+    <axis xyz="0 0 -1"/>
     <limit effort="1000.0" lower="0.0" upper="1.05" velocity="2.5"/>
   </joint>
   <joint name="right_external_rod_joint" type="revolute">
-    <mimic joint="right_finger_joint" multiplier="-1" offset="0"/>
+    <mimic joint="right_finger_joint" multiplier="1" offset="-1.05"/>
     <parent link="structure"/>
     <child link="right_external_rod"/>
@@ -241,5 +251,5 @@
   </joint>
   <joint name="right_fingertip_joint" type="revolute">
-    <mimic joint="right_finger_joint" multiplier="-1" offset="0"/>
+    <mimic joint="right_finger_joint" multiplier="1" offset="-1.05"/>
     <parent link="right_external_rod"/>
     <child link="right_finger_last_phalanx"/>
@@ -249,5 +259,5 @@
   </joint>
   <joint name="left_finger_joint" type="revolute">
-    <mimic joint="right_finger_joint" multiplier="-1" offset="0"/>
+    <mimic joint="right_finger_joint" multiplier="1" offset="-1.05"/>
     <parent link="structure"/>
     <child link="left_finger_first_phalanx"/>
@@ -257,5 +267,5 @@
   </joint>
   <joint name="left_external_rod_joint" type="revolute">
-    <mimic joint="right_finger_joint" multiplier="-1" offset="0"/>
+    <mimic joint="right_finger_joint" multiplier="1" offset="-1.05"/>
     <parent link="structure"/>
     <child link="left_external_rod"/>
@@ -265,5 +275,5 @@
   </joint>
   <joint name="left_fingertip_joint" type="revolute">
-    <mimic joint="right_finger_joint" multiplier="-1" offset="0"/>
+    <mimic joint="right_finger_joint" multiplier="1" offset="-1.05"/>
     <parent link="left_external_rod"/>
     <child link="left_finger_last_phalanx"/>
