Commit message: refactor: Cleanup explorer_hardware controller, arguments, launch files,...

File: explorer_description/gazebo/explorer.gazebo.xacro (robot description, xacro)
@@ -1,10 +1,16 @@
 <?xml version="1.0"?>
 <robot xmlns:xacro="http://ros.org/wiki/xacro">
-  <xacro:macro name="explorer_gazebo" params="">
-    <!-- ros_control plugin -->
+  <xacro:macro name="explorer_gazebo" params="use_ignition:=^|true">
     <gazebo>
-      <plugin filename="gz_ros2_control-system" name="gz_ros2_control::GazeboSimROS2ControlPlugin">
-        <parameters>$(find explorer_bringup)/config/explorer_controller.yaml</parameters>
-      </plugin>
+      <xacro:if value="${use_ignition}">
+        <plugin filename="gz_ros2_control-system" name="gz_ros2_control::GazeboSimROS2ControlPlugin">
+          <parameters>$(find explorer_bringup)/config/explorer_controller.yaml</parameters>
+        </plugin>
+      </xacro:if>
+      <xacro:unless value="${use_ignition}">
+        <plugin name="gazebo_ros2_control" filename="libgazebo_ros2_control.so">
+    <parameters>$(find explorer_bringup)/config/explorer_controller.yaml</parameters>
+  </plugin>
+      </xacro:unless>
     </gazebo>
     <gazebo reference="base_link">

File: explorer_description/ros2_control/explorer_actuators.ros2_control.xacro (robot description, xacro)
@@ -2,5 +2,5 @@
 <robot xmlns:xacro="http://www.ros.org/wiki/xacro">
   <xacro:include filename="$(find explorer_description)/urdf/explorer_joints.xacro" />
-  <xacro:macro name="explorer_ros2_control" params="name use_ignition:=^|false can_port:=^|vxcan1  host_id:=^|45 rt_stream_rate:=^|250 aux_stream_rate:=^|10">
+  <xacro:macro name="explorer_ros2_control" params="name can_port:=^|vxcan1  host_id:=^|45 rt_stream_rate:=^|250 aux_stream_rate:=^|10">
     <xacro:macro name="hw_intf_params">
       <plugin>orthopus_vesc_interface/VESCInterface</plugin>
@@ -54,15 +54,4 @@
     <xacro:explorer_gripper_servo_joint />
   </ros2_control>
-  <ros2_control name="${name}_gripper" type="system">
-    <hardware>
-      <!-- <xacro:if value="${use_ignition}">
-        <plugin>gz_ros2_control/GazeboSimSystem</plugin>
-      </xacro:if> -->
-      <xacro:unless value="${use_ignition}">
-        <plugin>explorer_hardware/RobotSystem</plugin>
-      </xacro:unless>
-    </hardware>
-    <xacro:explorer_gripper_joints />
-  </ros2_control>
   </xacro:macro>
 </robot>

File: explorer_description/ros2_control/explorer_simulation.ros2_control.xacro (robot description, xacro)
@@ -1,5 +1,5 @@
 <?xml version="1.0"?>
 <robot xmlns:xacro="http://www.ros.org/wiki/xacro">
-  <xacro:macro name="explorer_ros2_control" params="name use_ignition:=^|false can_port:=^|vxcan1 host_id:=^|45">
+  <xacro:macro name="explorer_ros2_control" params="name use_ignition:=^|true">
     <xacro:include filename="$(find explorer_description)/urdf/explorer_joints.xacro" />
     <ros2_control name="${name}" type="system">
@@ -9,5 +9,5 @@
         </xacro:if>
         <xacro:unless value="${use_ignition}">
-          <plugin>explorer_hardware/RobotSystem</plugin>
+          <plugin>gazebo_ros2_control/GazeboSystem</plugin>
         </xacro:unless>
       </hardware>
@@ -21,4 +21,7 @@
       <xacro:explorer_gripper_joints />
     </ros2_control>
+    <!-- Import Gazebo definitions + plugin -->
+      <xacro:include filename="$(find explorer_description)/gazebo/explorer.gazebo.xacro" />
+      <xacro:explorer_gazebo use_ignition="$(arg use_ignition)"/>
   </xacro:macro>
 </robot>

File: explorer_description/urdf/explorer.urdf.xacro (robot description, xacro)
@@ -1,11 +1,14 @@
 <?xml version="1.0"?>
 <robot xmlns:xacro="http://wiki.ros.org/xacro" name="explorer">
-  <xacro:arg name="use_ignition" default="false" />
-  <xacro:arg name="use_actuator_interface" default="false" />
-  <xacro:arg name="can_port" default="vxcan1" />
-  <xacro:arg name="host_id" default="45" />
-  <xacro:arg name="rt_stream_rate" default="250" />
-  <xacro:arg name="aux_stream_rate" default="50" />
   <xacro:arg name="use_POC2" default="false" />
+  <xacro:arg name="simulation" default="false" />
+    <!-- if Simulation-->
+    <xacro:arg name="use_ignition" default="true" />
+    <!-- else -->
+    <xacro:arg name="can_port" default="vxcan1" />
+    <xacro:arg name="host_id" default="45" />
+    <xacro:arg name="rt_stream_rate" default="250" />
+    <xacro:arg name="aux_stream_rate" default="50" />
+    <!-- endif -->
   <xacro:include filename="$(find gripper_pincette)/description/urdf/gripper_pincette_description.urdf.xacro"/>
   <!-- create link fixed to the "world" -->
@@ -60,13 +63,12 @@
   <xacro:gripper_pincette/>
   <!-- Import explorer ros2_control description -->
-  <xacro:unless value="$(arg use_actuator_interface)">
-    <xacro:include filename="$(find explorer_description)/ros2_control/explorer.ros2_control.xacro" />
+  <xacro:if value="$(arg simulation)">
+    <xacro:include filename="$(find explorer_description)/ros2_control/explorer_simulation.ros2_control.xacro" />
     <xacro:explorer_ros2_control name="explorer" use_ignition="$(arg use_ignition)" />
-  </xacro:unless>
-  <xacro:if value="$(arg use_actuator_interface)">
+  </xacro:if>
+  <xacro:unless value="$(arg simulation)">
     <xacro:include filename="$(find explorer_description)/ros2_control/explorer_actuators.ros2_control.xacro" />
     <xacro:explorer_ros2_control
       name="explorer"
-      use_ignition="$(arg use_ignition)"
       can_port="$(arg can_port)"
       host_id="$(arg host_id)"
@@ -74,9 +76,4 @@
       aux_stream_rate="$(arg aux_stream_rate)"
     />
-  </xacro:if>
-  <xacro:if value="$(arg use_ignition)">
-    <!-- Import Gazebo definitions + plugin -->
-    <xacro:include filename="$(find explorer_description)/gazebo/explorer.gazebo.xacro" />
-    <xacro:explorer_gazebo/>
-  </xacro:if>
+  </xacro:unless>
 </robot>

Commit message: [Simulation] 2nd yaml file for ros2 controller manager

File: explorer_description/gazebo/explorer.gazebo.xacro (robot description, xacro)
@@ -1,14 +1,22 @@
 <?xml version="1.0"?>
 <robot xmlns:xacro="http://ros.org/wiki/xacro">
-  <xacro:macro name="explorer_gazebo" params="use_ignition:=^|true">
+  <xacro:macro name="explorer_gazebo" params="use_ignition:=^|true extra_config:=''">
     <gazebo>
       <xacro:if value="${use_ignition}">
         <plugin filename="gz_ros2_control-system" name="gz_ros2_control::GazeboSimROS2ControlPlugin">
           <parameters>$(find explorer_bringup)/config/explorer_controller.yaml</parameters>
+          <xacro:property name="extra_config" value="$(arg extra_config)" />
+          <xacro:if value="${extra_config != ''}">
+            <parameters>${extra_config}</parameters>
+      </xacro:if>
         </plugin>
       </xacro:if>
       <xacro:unless value="${use_ignition}">
         <plugin name="gazebo_ros2_control" filename="libgazebo_ros2_control.so">
-    <parameters>$(find explorer_bringup)/config/explorer_controller.yaml</parameters>
+        <parameters>$(find explorer_bringup)/config/explorer_controller.yaml</parameters>
+        <xacro:property name="extra_config" value="$(arg extra_config)" />
+        <xacro:if value="${extra_config != ''}">
+                <parameters>${extra_config}</parameters>
+        </xacro:if>
   </plugin>
       </xacro:unless>

File: explorer_description/ros2_control/explorer_simulation.ros2_control.xacro (robot description, xacro)
@@ -1,5 +1,5 @@
 <?xml version="1.0"?>
 <robot xmlns:xacro="http://www.ros.org/wiki/xacro">
-  <xacro:macro name="explorer_ros2_control" params="name use_ignition:=^|true">
+  <xacro:macro name="explorer_ros2_control" params="name use_ignition:=^|true extra_config:=''">
     <xacro:include filename="$(find explorer_description)/urdf/explorer_joints.xacro" />
     <ros2_control name="${name}" type="system">
@@ -23,5 +23,5 @@
     <!-- Import Gazebo definitions + plugin -->
       <xacro:include filename="$(find explorer_description)/gazebo/explorer.gazebo.xacro" />
-      <xacro:explorer_gazebo use_ignition="$(arg use_ignition)"/>
+      <xacro:explorer_gazebo use_ignition="$(arg use_ignition)" extra_config="$(arg extra_config)"/>
   </xacro:macro>
 </robot>

File: explorer_description/urdf/explorer.urdf.xacro (robot description, xacro)
@@ -5,4 +5,5 @@
     <!-- if Simulation-->
     <xacro:arg name="use_ignition" default="true" />
+    <xacro:arg name="extra_config" default="" />
     <!-- else -->
     <xacro:arg name="can_port" default="vxcan1" />
@@ -80,5 +81,5 @@
   <xacro:if value="$(arg simulation)">
     <xacro:include filename="$(find explorer_description)/ros2_control/explorer_simulation.ros2_control.xacro" />
-    <xacro:explorer_ros2_control name="explorer" use_ignition="$(arg use_ignition)" />
+    <xacro:explorer_ros2_control name="explorer" use_ignition="$(arg use_ignition)" extra_config="$(arg extra_config)"/>
   </xacro:if>
   <xacro:unless value="$(arg simulation)">

Commit message: refactor: delete use_ignition param and always use latest Gazebo simulator

File: explorer_description/gazebo/explorer.gazebo.xacro (robot description, xacro)
@@ -1,16 +1,9 @@
 <?xml version="1.0"?>
 <robot xmlns:xacro="http://ros.org/wiki/xacro">
-  <xacro:macro name="explorer_gazebo" params="use_ignition:=^|true">
+  <xacro:macro name="explorer_gazebo">
     <gazebo>
-      <xacro:if value="${use_ignition}">
         <plugin filename="gz_ros2_control-system" name="gz_ros2_control::GazeboSimROS2ControlPlugin">
           <parameters>$(find explorer_bringup)/config/explorer_controller.yaml</parameters>
         </plugin>
-      </xacro:if>
-      <xacro:unless value="${use_ignition}">
-        <plugin name="gazebo_ros2_control" filename="libgazebo_ros2_control.so">
-    <parameters>$(find explorer_bringup)/config/explorer_controller.yaml</parameters>
-  </plugin>
-      </xacro:unless>
     </gazebo>
     <gazebo reference="base_link">

File: explorer_description/ros2_control/explorer_simulation.ros2_control.xacro (robot description, xacro)
@@ -1,14 +1,9 @@
 <?xml version="1.0"?>
 <robot xmlns:xacro="http://www.ros.org/wiki/xacro">
-  <xacro:macro name="explorer_ros2_control" params="name use_ignition:=^|true">
+  <xacro:macro name="explorer_ros2_control" params="name">
     <xacro:include filename="$(find explorer_description)/urdf/explorer_joints.xacro" />
     <ros2_control name="${name}" type="system">
       <hardware>
-        <xacro:if value="${use_ignition}">
-          <plugin>gz_ros2_control/GazeboSimSystem</plugin>
-        </xacro:if>
-        <xacro:unless value="${use_ignition}">
-          <plugin>gazebo_ros2_control/GazeboSystem</plugin>
-        </xacro:unless>
+        <plugin>gz_ros2_control/GazeboSimSystem</plugin>
       </hardware>
       <xacro:explorer_joint_1 />
@@ -23,5 +18,5 @@
     <!-- Import Gazebo definitions + plugin -->
       <xacro:include filename="$(find explorer_description)/gazebo/explorer.gazebo.xacro" />
-      <xacro:explorer_gazebo use_ignition="$(arg use_ignition)"/>
+      <xacro:explorer_gazebo/>
   </xacro:macro>
 </robot>

File: explorer_description/urdf/explorer.urdf.xacro (robot description, xacro)
@@ -4,5 +4,4 @@
   <xacro:arg name="simulation" default="false" />
     <!-- if Simulation-->
-    <xacro:arg name="use_ignition" default="true" />
     <!-- else -->
     <xacro:arg name="can_port" default="vxcan1" />
@@ -80,5 +79,5 @@
   <xacro:if value="$(arg simulation)">
     <xacro:include filename="$(find explorer_description)/ros2_control/explorer_simulation.ros2_control.xacro" />
-    <xacro:explorer_ros2_control name="explorer" use_ignition="$(arg use_ignition)" />
+    <xacro:explorer_ros2_control name="explorer"/>
   </xacro:if>
   <xacro:unless value="$(arg simulation)">

Commit message: dev: Add effort interface to urdf files + add controller type (custom / controller)

File: explorer_description/gazebo/explorer.gazebo.xacro (robot description, xacro)
@@ -1,9 +1,9 @@
 <?xml version="1.0"?>
 <robot xmlns:xacro="http://ros.org/wiki/xacro">
-  <xacro:macro name="explorer_gazebo" params="use_ignition:=^|true">
+  <xacro:macro name="explorer_gazebo" params="use_ignition:=^|true robot_controller_config">
     <gazebo>
       <xacro:if value="${use_ignition}">
         <plugin filename="gz_ros2_control-system" name="gz_ros2_control::GazeboSimROS2ControlPlugin">
-          <parameters>$(find explorer_bringup)/config/explorer_controller.yaml</parameters>
+          <parameters>$(find explorer_bringup)/config/explorer_${robot_controller_config}.yaml</parameters>
         </plugin>
       </xacro:if>

File: explorer_description/ros2_control/explorer_simulation.ros2_control.xacro (robot description, xacro)
@@ -1,5 +1,5 @@
 <?xml version="1.0"?>
 <robot xmlns:xacro="http://www.ros.org/wiki/xacro">
-  <xacro:macro name="explorer_ros2_control" params="name use_ignition:=^|true">
+  <xacro:macro name="explorer_ros2_control" params="name use_ignition:=^|true robot_controller_config">
     <xacro:include filename="$(find explorer_description)/urdf/explorer_joints.xacro" />
     <ros2_control name="${name}" type="system">
@@ -23,5 +23,5 @@
     <!-- Import Gazebo definitions + plugin -->
       <xacro:include filename="$(find explorer_description)/gazebo/explorer.gazebo.xacro" />
-      <xacro:explorer_gazebo use_ignition="$(arg use_ignition)"/>
+      <xacro:explorer_gazebo use_ignition="$(arg use_ignition)" robot_controller_config="$(arg robot_controller_config)"/>
   </xacro:macro>
 </robot>

File: explorer_description/urdf/explorer.urdf.xacro (robot description, xacro)
@@ -3,4 +3,5 @@
   <xacro:arg name="use_POC2" default="false" />
   <xacro:arg name="simulation" default="false" />
+  <xacro:arg name="robot_controller_config" default="controller" />
     <!-- if Simulation-->
     <xacro:arg name="use_ignition" default="true" />
@@ -80,5 +81,5 @@
   <xacro:if value="$(arg simulation)">
     <xacro:include filename="$(find explorer_description)/ros2_control/explorer_simulation.ros2_control.xacro" />
-    <xacro:explorer_ros2_control name="explorer" use_ignition="$(arg use_ignition)" />
+    <xacro:explorer_ros2_control name="explorer" use_ignition="$(arg use_ignition)" robot_controller_config="$(arg robot_controller_config)"/>
   </xacro:if>
   <xacro:unless value="$(arg simulation)">

File: explorer_description/urdf/explorer_joints.xacro (robot description, xacro)
@@ -3,4 +3,8 @@
     <xacro:macro name="explorer_joint_1">
       <joint name="joint_1">
+        <command_interface name="effort">
+          <param name="min">-100</param>
+          <param name="max">100</param>
+        </command_interface>
         <command_interface name="position">
           <param name="min">-2*{pi}</param>
@@ -20,4 +24,8 @@
     <xacro:macro name="explorer_joint_2">
       <joint name="joint_2">
+        <command_interface name="effort">
+          <param name="min">-100</param>
+          <param name="max">100</param>
+        </command_interface>
         <command_interface name="position">
           <param name="min">-2*{pi}</param>
@@ -37,4 +45,8 @@
     <xacro:macro name="explorer_joint_3">
       <joint name="joint_3">
+        <command_interface name="effort">
+          <param name="min">-100</param>
+          <param name="max">100</param>
+        </command_interface>
         <command_interface name="position">
           <param name="min">{-pi}</param>
@@ -54,4 +66,8 @@
     <xacro:macro name="explorer_joint_4">
       <joint name="joint_4">
+        <command_interface name="effort">
+          <param name="min">-100</param>
+          <param name="max">100</param>
+        </command_interface>
         <command_interface name="position">
           <param name="min">-2*{pi}</param>
@@ -71,4 +87,8 @@
     <xacro:macro name="explorer_joint_5">
       <joint name="joint_5">
+        <command_interface name="effort">
+          <param name="min">-100</param>
+          <param name="max">100</param>
+        </command_interface>
         <command_interface name="position">
           <param name="min">-2*{pi}</param>
@@ -88,4 +108,8 @@
     <xacro:macro name="explorer_joint_6">
       <joint name="joint_6">
+        <command_interface name="effort">
+          <param name="min">-100</param>
+          <param name="max">100</param>
+        </command_interface>
         <command_interface name="position">
           <param name="min">-2*{pi}</param>
